File: schematics/Control_Unit/Control_Unit.sch (EAGLE design)
At the start: 170 parts, among them IC1 74HC174N, IC10 74HC74N, IC100 74HCT32N, IC101 74HCT08N, IC102 74HCT32N, IC103 74HC373N, IC104 74HCT08N, IC105 74HCT04N, IC106 74HCT32N, IC107 74HCT08N, IC108 74HCT32N, IC109 74HCT08N, IC11 74HC74N, IC110 74HCT32N, IC111 74HCT08N, IC112 74HCT08N, IC113 74HCT08N, IC114 74HCT08N, IC117 74HCT32N, IC118 74HCT32N, IC12 74AC08N, IC121 74HCT04N, IC122 74HCT04N, IC123 74HCT04N, IC124 74HCT32N, IC125 74HCT08N, IC126 74AC157N, IC127 74HCT08N, IC128 74AC08N, IC129 74AC08N, IC13 74AC08N, IC130 74HCT04N, IC14 74HC74N, IC15 74HC74N, IC16 74AC08N, IC164 74HC174N, IC165 74HC174N, IC166 74HC174N, IC167 74HC174N, IC168 74HCT32N, IC169 74HCT32N, IC17 74HCT32N, IC172 74HCT32N, IC173 74HCT32N, IC174 74HCT32N, IC175 74HC193N, IC176 74HC193N, IC177 74HC193N, IC178 74HC193N, IC179 74HC193N, IC18 74AC08N, IC180 74HC193N, IC181 74HC193N, IC182 74HC193N, IC19 74AC08N, IC190 74HCT32N, IC191 74HCT32N, IC2 74HC174N, IC20 74AC08N, IC21 74AC08N, IC22 74HCT32N, IC23 74HCT08N, IC24 74HCT08N, IC25 74HCT32N, IC26 74HCT08N, IC27 74HCT08N, IC28 74HCT08N, IC29 74HCT08N, IC3 74HC151N, IC30 74HCT08N, IC31 74HCT08N, IC32 74HCT32N, IC33 74HCT04N, IC34 74HCT08N, IC35 74HCT04N, IC36 CY62256LL-PC, IC37 74HCT04N, IC38 74HCT08N, IC39 74HCT08N, IC4 74HC174N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

Commit message: clean up schematic. next up is Instruction fetch & decode
Parts:
- removed IC100, IC102, IC106, IC117, IC118, IC17, IC54, IC64, IC70, IC73, IC80, IC81, IC94: 74HCT32N, 74xx-eu:74HCT32N
- removed IC105, IC121, IC122, IC123, IC91, IC95, IC97, IC98: 74HCT04N, 74xx-eu:74HCT04N
- removed IC107, IC109, IC111, IC112, IC113, IC114, IC45, IC48, IC51, IC53, IC85, IC90, IC92: 74HCT08N, 74xx-eu:74HCT08N
- IC33: value 74HCT04N -> 74HCT32N; device 74xx-eu:74HCT04N -> 74xx-eu:74HCT32N
Connections:
- net CLR_NOT_CS_LDA renamed CLR_NOT_CS_LDR
- net CONNECT_BR_TO_ABUS/CLR_NOT_OE_LDA renamed CONNECT_PTR_TO_ABUS/CLR_NOT_OE_LDR
- net CONNECT_BR_TO_ABUS_STR/CONNECT_REG_TO_DBUS_STR/CLR_NOT_WE_STR/SELECTOR_TABLE_2 renamed CONNECT_PTR_TO_ABUS_STR/CONNECT_REG_TO_DBUS_STR/CLR_NOT_WE_STR/SELECTOR_TABLE_2
- net FILL_REGISTER_LDA renamed FILL_REGISTER_LDR
- net ALU_CARRY_OUT: now also IC101B.I0, IC127A.I0; no longer IC112D.I0, IC92D.I0
- net ALU_NR1_ENABLE_ALU: now also IC33C.I0; no longer IC117A.I0
- net ALU_NR1_ENABLE_JMP_O_PTR_ADD: now also IC33C.I1; no longer IC117A.I1
- net ALU_NR2_ENABLE_ALU: now also IC33B.I0; no longer IC118A.I0
- net ALU_NR2_ENABLE_JMP_O_PTR_ADD: now also IC33B.I1; no longer IC118A.I1
- net DATA0: now also IC82A.A
- net DATA1: now also IC82A.B
- net DATA2: now also IC82A.C
- net DATA3: now also IC82A.D
- net DATA4: now also IC83A.A
- net DATA5: now also IC83A.B
- net DATA6: now also IC83A.C
- net DATA7: now also IC83A.D
- net DBUS_SELECTOR_TABLE_2: now also IC33D.I0; no longer IC52D.I0
- net FILL_PC_L_JMP_O: now also IC38D.O; no longer IC51D.O
- net FILL_PTR_L_PTR_ADD: now also IC104C.O; no longer IC109D.O
- net FILL_REGISTER_ALU/ALU_TO_DBUS: now also IC110A.I0; no longer IC81B.I0
- net FILL_REGISTER_MOV: now also IC190B.I0; no longer IC174D.I0
- net GND: no longer IC82A.A, IC82A.B, IC82A.C, IC82A.D
- net INPUT_REG0: now also IC124A.I0; no longer IC17B.I0
- net IR_DATA_OUT_7: now also IC104B.I0, IC125A.I0, IC130D.I, IC130F.I; no longer IC114D.I0, IC121B.I, IC85D.I0, IC91B.I
- net LATCH_ALU_INPUT_B_ALU: now also IC110D.I0, IC190D.I0; no longer IC54D.I0, IC73B.I0
- net LATCH_ALU_INPUT_B_JMP_O: now also IC38A.O, IC99B.I0; no longer IC106B.I0, IC45D.O
- net LATCH_ALU_INPUT_B_PTR_ADD: now also IC173D.I0, IC99B.I1; no longer IC102A.I0, IC106B.I1
- net N$101: now also IC110C.I1; no longer IC80B.I1
- net N$11: now also IC33A.O, IC52D.I1; no longer IC64B.O, IC70B.I1
- net N$110: now also IC190D.I1; no longer IC54D.I1
- net N$113: now also IC191D.I0; no longer IC174A.I0
- net N$115: now also IC110C.O; no longer IC80B.O
- net N$128: now also IC101D.I0, IC130D.O; no longer IC90D.I0, IC91B.O
- net N$131: now also IC47E.I; no longer IC44B.I
- net N$132: now also IC101A.I1, IC38A.I1, IC38B.I1, IC38D.I1; no longer IC45D.I1, IC48D.I1, IC51D.I1, IC53D.I1
- net N$133: now also IC93C.O; no longer IC98B.O
- net N$135: now also IC110A.O; no longer IC81B.O
- net N$137: now also IC101A.O, IC101B.I1; no longer IC53D.O, IC92D.I1
- net N$139: now also IC101B.O, IC101D.I1, IC104B.I1; no longer IC85D.I1, IC90D.I1, IC92D.O
- net N$140: now also IC93E.I; no longer IC97B.I
- net N$141: now also IC93A.I, IC99A.O; no longer IC94C.O, IC95B.I
- net N$142: now also IC99A.I0; no longer IC94C.I0
- net N$143: now also IC108C.O; no longer IC100B.O
- net N$144: now also IC93C.I; no longer IC98B.I
- net N$145: now also IC93E.O; no longer IC97B.O
- net N$147: now also IC110A.I1; no longer IC81B.I1
- net N$149: now also IC104A.I1, IC104C.I1, IC127B.I1; no longer IC107D.I1, IC109D.I1, IC111D.I1
- net N$151: now also IC173D.I1; no longer IC102A.I1
- net N$152: now also IC110D.I1, IC99B.O; no longer IC106B.O, IC73B.I1
- net N$153: now also IC127A.I1, IC127B.O; no longer IC111D.O, IC112D.I1
- net N$155: now also IC108C.I0; no longer IC100B.I0
- net N$158: now also IC125A.O, IC93F.I; no longer IC114D.O, IC123B.I
- net N$159: now also IC125A.I1, IC127A.O, IC127D.I1; no longer IC112D.O, IC113D.I1, IC114D.I1
- net N$161: now also IC127D.I0, IC130F.O; no longer IC113D.I0, IC121B.O
- net N$162: now also IC127D.O, IC93D.I; no longer IC113D.O, IC122B.I
- net N$167: now also IC33B.O; no longer IC118A.O
- net N$197: now also IC124C.I0; no longer IC174C.I0
- net N$198: now also IC124C.I1; no longer IC174C.I1
- net N$2: now also IC33D.O, IC52D.I0; no longer IC52D.O, IC70B.I0
- net N$202: now also IC33C.O; no longer IC117A.O
- net N$21: now also IC130C.I; no longer IC105E.I
- net N$22: now also IC130B.O; no longer IC33A.O
- net N$240: now also IC93A.O; no longer IC95B.O
- net N$51: now also IC49A.O; no longer IC49C.O
- net N$55: now also IC191D.O; no longer IC174A.O
- net N$56: now also IC190B.I1; no longer IC174D.I1
- net N$7: now also IC124C.O; no longer IC174C.O
- net N$8: now also IC191D.I1; no longer IC174A.I1
- net N$82: now also IC124A.O, IC130B.I; no longer IC17B.O, IC33A.I
- net N$90: now also IC52D.O; no longer IC70B.O
- net N$94: now also IC165A.D3
- net N$96: now also IC110D.O; no longer IC73B.O
- net OPCODE_5: now also IC49A.I0; no longer IC49C.I0
- net OPCODE_7: now also IC49A.I1; no longer IC49C.I1
- net OPERAND_REGB_OUTPUT: now also IC33D.I1; no longer IC52D.I1
- net OUTPUT_REG0_JMP: now also IC124A.I1; no longer IC17B.I1
- net PC_H_COUNT_DOWN_JMP_O: now also IC104B.O; no longer IC85D.O
- net PC_H_COUNT_UP_JMP_O: now also IC101D.O, IC99A.I1; no longer IC90D.O, IC94C.I1
- net PTR_HIGH_COUNT_DOWN: now also IC93F.O; no longer IC123B.O
- net PTR_HIGH_COUNT_UP: now also IC93D.O; no longer IC122B.O
- net REG1_ZERO: now also IC130C.O; no longer IC105E.O
- net SP_COUNT_UP: now also IC47E.O; no longer IC44B.O
- net STATE_2: now also IC38A.I0; no longer IC45D.I0
- net STATE_3: now also IC104A.I0, IC38B.I0; no longer IC107D.I0, IC48D.I0
- net STATE_4: now also IC104C.I0, IC38D.I0; no longer IC109D.I0, IC51D.I0
- net STATE_5: now also IC101A.I0, IC127B.I0; no longer IC111D.I0, IC53D.I0
- net WRITE_PC_L_ALU_LATCH_JMP_O: now also IC110C.I0; no longer IC80B.I0
- net WRITE_PTR_L_TO_DBUS_PTR_ADD: now also IC173D.O, IC33A.I1; no longer IC102A.O, IC64B.I1
- net WRITE_REGB_TO_DBUS_JMP: now also IC108C.I1; no longer IC100B.I1
- net WRITE_REGB_TO_DBUS_JMP_O: now also IC38B.O; no longer IC48D.O
- net WRITE_REGB_TO_DBUS_PTR_ADD: now also IC104A.O; no longer IC107D.O
- net WRITE_REG_TO_DBUS_ALU: now also IC190D.O; no longer IC54D.O
- net WRITE_REG_TO_DBUS_JMP_O: now also IC33A.I0; no longer IC64B.I0
- net WRITE_REG_TO_DBUS_MOV: now also IC190B.O; no longer IC174D.O
Other:
- note added: "Instruction Fetch and Decode"
- note added: "LDR"
- note added: "Probalby need to latch it at the same time as ALU_LATCH"
- note added: "SP never needs to load input. It just gets reseted on startup"
- note removed: "LDA"
- note removed: "Probalby need to latch it!"
- note removed: "SP never needs to load input. I just gets reseted on startup"
- moved on the sheet: IC108B, IC10A, IC10B, IC11A, IC11B, IC126, IC128A, IC128B, IC128C, IC128D, IC129A, IC129B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

Commit message: add fetch cycle
Parts:
- added IC17, IC51: 74HCT32N, 74xx-eu:74HCT32N
- added IC45, IC48: 74HCT04N, 74xx-eu:74HCT04N
Connections:
- removed net CNNCT_PC_ABUS/CLR_NOT_OE/CLR_NOT_CS_CYCL_0: IC10A.Q, IC10B.D
- removed net IR_LOAD_INPUT/CLR_NOT_CS_CYCL_2: IC10B.Q, IC11A.D
- removed net IR_LOW_LOAD_INPUT: IC50A.CLK, IC6A.CLK
- new net CLR_NOT_OE/CLR_NOT_CS_CYCL_0: IC17A.I0, IC17D.I0, IC51D.O
- new net N$163: IC10A.Q, IC10B.D, IC51D.I1
- new net N$31: IC34D.O, IC48F.I
- new net N$98: IC17D.O, IC37B.I
- new net N$99: IC45F.O, IC96G$1.!CE
- new net OPCODE_LOAD_INPUT: IC10B.Q, IC11A.D, IC50A.CLK, IC51D.I0, IC6A.CLK
- net CLR_NOT_CS_STR: now also IC17A.I1; no longer IC63D.I0
- net CONNECT_PTR_TO_ABUS/CLR_NOT_OE_LDR: now also IC17D.I1; no longer IC37B.I
- net MEM_NOT_CE: now also IC63D.O; no longer IC37A.O
- net N$126: now also IC17A.O, IC63D.I0; no longer IC37A.I, IC63D.O
- net N$69: now also IC36G$1.!CE, IC48F.O; no longer IC34C.O, IC96G$1.!CE
- net N$70: now also IC34C.O, IC45F.I; no longer IC34D.O, IC36G$1.!CE
Other:
- note added: "Addr15 goes to Enable of the mem chips"
- note removed: "TheAddr15 line goes to Enable of the mem chips"
- moved on the sheet: IC34C, IC34D, IC35F, IC63D

Commit message: fix offset commands JMP and ADD_PTR
Parts:
- added IC53: 74HCT32N, 74xx-eu:74HCT32N
- added IC54: 74HCT04N, 74xx-eu:74HCT04N
- added IC64, IC70: 74HCT08N, 74xx-eu:74HCT08N
- IC31: value 74HCT08N -> 74HCT04N; device 74xx-eu:74HCT08N -> 74xx-eu:74HCT04N
Connections:
- removed net N$15 (its old number): IC124B.I0, IC20B.O, IC31C.I1
- new net N$100: IC53A.O, IC54D.I
- new net N$168: IC53A.I1
- new net N$194: IC20D.O
- new net PC_COUNT_UP_FETCH1: IC53A.I0
- net INPUT_REG0: now also IC64C.I0; no longer IC124A.I0
- net N$132: now also IC124B.I1, IC70C.O; no longer IC31C.O
- net N$149: now also IC29C.I1, IC31A.O; no longer IC101C.I1, IC104A.I1, IC104C.I1, IC104D.I1, IC124B.I1, IC127B.I1, IC20C.O
- net N$22: now also IC31A.I, IC64C.O, IC70C.I1; no longer IC130B.O, IC31C.I0
- net N$7: now also IC101C.I1, IC104A.I1, IC104C.I1, IC104D.I1, IC124B.I0, IC127B.I1, IC20B.O; no longer IC124C.O, IC29C.I0
- net N$82: now also IC124C.O, IC29C.I0, IC70C.I0; no longer IC124A.O, IC130B.I, IC29C.I1
- net N$97: now also IC20C.O; no longer IC20D.O
- net OUTPUT_REG0_JMP: now also IC64C.I1; no longer IC124A.I1
- net PC_COUNT_UP: now also IC54D.O
Other:
- note added: "SAVE_LR/RET"
- moved on the sheet: IC124B, IC125C, IC127C, IC130A, IC169A, IC172A, IC172B, IC172C, IC172D, IC173A, IC173B, IC173C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
