File: schematics/Control_Unit/Control_Unit.sch (EAGLE design)
At the start: 245 parts, among them IC1 74HCT32N, IC10 74HC74N, IC100 74HCT374N, IC101 74HCT08N, IC102 74HC151N, IC103 74HC373N, IC105 74HC151N, IC106 74HC151N, IC108 74HCT32N, IC11 74HC74N, IC110 74HCT32N, IC111 74HC151N, IC112 74HCT32N, IC113 74HC151N, IC114 74HC151N, IC115 74HC151N, IC116 74HC373N, IC117 74HC74N, IC12 74AC08N, IC124 74HCT32N, IC125 74HCT08N, IC126 74AC157N, IC127 74HCT08N, IC128 74AC08N, IC129 74AC08N, IC13 74AC08N, IC134 74HCT08N, IC135 74HCT08N, IC136 74HCT08N, IC14 74HC74N, IC141 74HCT32N, IC15 74HC74N, IC16 74AC08N, IC168 74HCT32N, IC169 74HCT32N, IC17 74HCT32N, IC172 74HCT32N, IC173 74HCT32N, IC175 74HC193N, IC176 74HC193N, IC177 74HC193N, IC178 74HC193N, IC179 74HC193N, IC18 74AC08N, IC180 74HC193N, IC181 74HC193N, IC182 74HC193N, IC19 74AC08N, IC190 74HCT32N, IC191 74HCT32N, IC2 74HCT32N, IC20 74AC08N, IC21 74AC08N, IC22 74HCT32N, IC23 74HCT08N, IC24 74HCT08N, IC25 74HCT32N, IC26 74HCT08N, IC27 74HCT08N, IC28 74HCT08N, IC29 74HCT32N, IC3 74HC151N, IC30 74HCT08N, IC31 74HCT00N, IC32 74HCT32N, IC33 74HCT32N, IC34 74HCT08N, IC35 74HCT04N, IC36 74HCT32N, IC38 74HCT08N, IC39 74HCT08N, IC40 74HCT08N, IC41 74HCT08N, IC42 74HC373N, IC43 74HCT04N, IC44 74ACT157N, IC46 74ACT157N, IC47 74HCT04N, IC48 74ACT02N, IC49 74AC86N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

Commit message: forgot it
Parts:
- removed C156: (no value), rcl:C-EU025-025X050
Connections:
- net ADRR_15: now also IC17C.I0; no longer IC25C.I0
- net FILL_PC_H_RET: now also IC1A.I0; no longer IC17D.I0
- net FILL_PC_L_JMP_O: now also IC1D.I0; no longer IC80C.I0
- net FILL_PC_L_RET: now also IC1D.I1; no longer IC80C.I1
- net GND: no longer C156.2
- net MEM_NOT_CE: now also IC17C.I1, IC17D.I1; no longer IC25C.I1, IC36A.I1
- net N$12: now also IC49D.I1; no longer IC49D.I0
- net N$163: now also IC1D.O; no longer IC80C.O
- net N$171: now also IC36B.O; no longer IC17C.O
- net N$31: now also IC17D.O; no longer IC36A.O
- net N$32: now also IC1C.O; no longer IC36B.O
- net N$33: now also IC1A.O; no longer IC17D.O
- net N$67: now also IC17D.I0; no longer IC36A.I0
- net N$70: now also IC17C.O; no longer IC25C.O
- net PC_H_LOAD_INPUT_TABLE_1: now also IC1A.I1; no longer IC17D.I1
- net PC_LOW_LOAD_INPUT_JMP: now also IC1C.I0; no longer IC36B.I0
- net PC_L_LOAD_INPUT_TABLE_1: now also IC1C.I1; no longer IC36B.I1
- net VCC: now also IC49D.I0; no longer C156.1, IC49D.I1
- net WRITE_LR_H_DBUS_RET: now also IC36B.I0; no longer IC17C.I0
- net WRITE_PC_L_DBUS_SAVE_LR: now also IC36B.I1; no longer IC17C.I1
Other:
- moved on the sheet: C100, C101, C110, C111, C112, C113, C114, C115, C116, C118, C126, C127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

Commit message: regroup
Connections:
- net CONNECT_PTR_TO_ABUS/CLR_NOT_OE_LDR: now also IC36A.I0; no longer IC25B.I0
- net CONNECT_PTR_TO_ABUS/CONNECT_REG_TO_DBUS/CLR_NOT_WE/SELECTOR_TABLE_2_STR: now also IC36A.I1; no longer IC25B.I1
- net N$190: now also IC80C.I1; no longer IC25A.I1
- net N$192: now also IC80C.I0; no longer IC25A.I0
- net N$193: now also IC80C.O; no longer IC25A.O
- net PTR_TO_ABUS/!PC_TO_ABUS: now also IC36A.O; no longer IC25B.O
Other:
- moved on the sheet: IC117B, IC136A, IC172C, IC40A, IC43D, IC75A

Commit message: optimize chip count :)
Parts:
- removed IC25: 74HCT32N, 74xx-eu:74HCT32N
- removed IC54: 74ACT02N, 74xx-eu:74ACT02N
Connections:
- removed net INPUT_REG0: IC126A.1B, IC129A.O, IC135A.I0, IC135B.I0, IC30A.I0, IC31B.I0, IC41A.I0, IC41B.I0
- removed net N$201: IC54D.O, IC80A.I0
- removed net N$217: IC108D.O, IC48D.I0
- removed net N$224: IC136A.I1, IC136D.I0, IC34B.O
- removed net N$227: IC169B.I1, IC48D.O
- removed net N$247: IC136C.I1, IC136D.I1, IC43D.O
- removed net N$54: IC34B.I0, IC43E.O
- removed net N$84: IC128B.O, IC76B.I1
- removed net N$85: IC128C.O, IC76C.I1
- removed net N$86: IC128D.O, IC76D.I1
- removed net OUTPUT_REG0_JMP: IC128A.O, IC31B.I1, IC76A.I1
- new net INPUT_REG0/OPCODE_5/OPCODE_4_IS_NULL: IC126A.1B, IC129A.O, IC135A.I0, IC135B.I0, IC30A.I0, IC34A.I0, IC40B.I1, IC41A.I0, IC41B.I0
- new net INPUT_REG_IS_OUTPUT_REG: IC40C.I0, IC43E.O
- new net N$45: IC40C.I1, IC80A.O
- new net OPC_67_OUPUT0/REG0_JMP: IC128A.O, IC136A.I0, IC34A.I1, IC76A.I1
- new net OPC_67_OUPUT1: IC128B.O, IC136B.I0, IC76B.I1
- new net OPC_67_OUPUT2: IC128C.O, IC136C.I0, IC76C.I1
- new net OPC_67_OUPUT3: IC128D.O, IC136D.I0, IC76D.I1
- net CLR_NOT_CS_POP: now also IC48D.I0; no longer IC54A.I0
- net CLR_NOT_OE_POP: now also IC48D.O; no longer IC54A.O
- net FILL_REGISTER_ALU/ALU_TO_DBUS: now also IC169B.I0; no longer IC54C.I0
- net INPUT_REG_IS_NOT_OUTPUT_REG: now also IC43E.I; no longer IC48D.I1, IC54D.I0
- net N$12: now also IC40D.O; no longer IC34C.O
- net N$14: now also IC43D.O; no longer IC54C.O
- net N$147: now also IC169B.I1; no longer IC54C.I1
- net N$149: now also IC47F.O; no longer IC31B.O, IC47F.I
- net N$157: now also IC48D.I1; no longer IC54A.I1
- net N$18: now also IC169B.O, IC43D.I; no longer IC136B.I1, IC136C.I0, IC34A.O
- net N$185: now also IC108D.I1; no longer IC25D.I1
- net N$187: now also IC108D.I0; no longer IC25D.I0
- net N$20: now also IC108D.O; no longer IC25D.O
- net N$203: now also IC40B.O; no longer IC169B.O
- net N$206: now also IC80A.I0; no longer IC54D.I1
- net N$21: now also IC40B.I0; no longer IC169B.I0
- net N$22: now also IC34A.O, IC47F.I; no longer IC47F.O
- net N$266: now also IC40D.I1; no longer IC34C.I1
- net N$53: now also IC136A.I1, IC136B.I1, IC136C.I1, IC136D.I1; no longer IC34A.I1, IC34B.I1
- net OPCODE_4: no longer IC108D.I0
- net OPCODE_5: no longer IC108D.I1
- net OPCODE_6: no longer IC34A.I0, IC43E.I
- net OPCODE_7: no longer IC136A.I0, IC136B.I0, IC43D.I
- net REGISTER_OUTPUT_SEL_3: now also IC40D.I0; no longer IC34C.I0
- net TWO_BYTE_CMD: now also IC40C.O; no longer IC80A.O
Other:
- moved on the sheet: IC108B, IC108D, IC124C, IC124D, IC125B, IC125D, IC169B, IC34A, IC43D, IC43E, IC47F, IC48D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

Commit message: start routing
Parts:
- removed C115, C81, C92: (no value), rcl:C-EUC1206
- removed IC76: 74HCT08N, 74xx-eu:74HCT08N
- added IC4: 74AC08N, 74xx-eu:74AC08N
Connections:
- removed net OUTPUT_REG0: IC126A.1A, IC76A.O
- removed net OUTPUT_REG1: IC126A.2A, IC76B.O
- removed net OUTPUT_REG2: IC126A.3A, IC76C.O
- removed net OUTPUT_REG3: IC126A.4A, IC76D.O
- new net N$24: IC126A.4A, IC4D.O
- new net N$27: IC126A.3A, IC4C.O
- new net N$69: IC126A.2A, IC4B.O
- new net N$72: IC126A.1A, IC4A.O
- net GND: no longer C115.2, C81.2, C92.2
- net INPUT_REG_IS_NOT_OUTPUT_REG: now also IC4A.I0, IC4B.I0, IC4C.I0, IC4D.I0; no longer IC76A.I0, IC76B.I0, IC76C.I0, IC76D.I0
- net N$219: now also IC31B.O; no longer IC34D.O
- net N$44: now also IC31B.I0; no longer IC34D.I1
- net OPCODE_5: now also IC31B.I1; no longer IC35E.I
- net OPC_67_OUPUT0/REG0_JMP: now also IC4A.I1; no longer IC76A.I1
- net OPC_67_OUPUT1: now also IC4B.I1; no longer IC76B.I1
- net OPC_67_OUPUT2: now also IC4C.I1; no longer IC76C.I1
- net OPC_67_OUPUT3: now also IC4D.I1; no longer IC76D.I1
- net SAVE_LR/RET: now also IC35E.I; no longer IC34D.I0
- net VCC: no longer C115.1, C81.1, C92.1
Other:
- moved on the sheet: C116, C117, C118, C120, C121, C122, C123, C124, C126, C127, C129, C130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

Commit message: fix. gonna try to reduce cycles to 8 per instruction now
Parts:
- removed IC134, IC40: 74HCT08N, 74xx-eu:74HCT08N
- removed IC2, IC32: 74HCT32N, 74xx-eu:74HCT32N
- removed JP6: (no value), pinhead:PINHD-1X2
- added IC5, IC8: 74ACT02N, 74xx-eu:74ACT02N
- added IC6, IC7: 74HC193N, custom_parts:74HC193N
Connections:
- net ALU_NR3_ENABLE renamed ALU_NR3_ENABLE_ALU
- net ALU_NR4_ENABLE renamed ALU_NR4_ENABLE_ALU
- removed net INPUT_REG_IS_OUTPUT_REG: IC40C.I0, IC43E.O
- removed net N$128: IC101B.I0, IC49C.O
- removed net N$144: IC181A.DN, IC75C.O
- removed net N$145: IC180A.BO, IC75C.I1
- removed net N$164: IC127C.I0, IC47E.O
- removed net N$206: IC108A.O, IC80A.I0
- removed net N$222: IC129A.I1, IC129B.I1, IC43C.O
- removed net N$242: IC179A.BO, IC180A.DN
- removed net N$44: IC31B.I0, IC35E.O
- removed net NOT_USED2: IC134A.O
- removed net NOT_USED3: IC134B.O
- removed net NOT_USED4: IC134C.O
- removed net NOT_USED5: IC134D.O
- new net !IR_DATA_OUT_7: IC101D.I0, IC127C.I0, IC36D.I0, IC47E.O
- new net !OPCODE_5: IC129A.I1, IC129B.I1, IC43C.O, IC75C.I1
- new net N$77: IC6A.CO, IC7A.UP
- new net N$80: IC112A.O, IC80C.I0
- new net TIMER_CLOCK: IC6A.UP, JP1.3
- new net TIMER_REG_0: IC115A.D7, IC6A.QA
- new net TIMER_REG_1: IC114A.D7, IC6A.QB
- new net TIMER_REG_2: IC113A.D7, IC6A.QC
- new net TIMER_REG_3: IC111A.D7, IC6A.QD
- new net TIMER_REG_4: IC106A.D7, IC7A.QA
- new net TIMER_REG_5: IC105A.D7, IC7A.QB
- new net TIMER_REG_6: IC7A.QC, IC98A.D7
- new net TIMER_REG_7: IC102A.D7, IC7A.QD
- new net UNUSED: IC34B.O
- net !REGISTER_RESET: now also IC6A.CLR, IC7A.CLR
- net ALU_CARRY_BIT: now also IC34D.I0, JP1.16; no longer IC40A.I0, JP1.7
- net ALU_CARRY_IN: now also IC34D.O; no longer IC40A.O
- net ALU_CARRY_OUT: now also IC101C.I0; no longer IC101D.I0
- net DATA0: now also IC77A.1A; no longer IC77A.1B
- net DATA1: now also IC77A.2A; no longer IC77A.2B
- net DATA2: now also IC77A.3A; no longer IC77A.3B
- net DATA3: now also IC77A.4A; no longer IC77A.4B
- net DATA4: now also IC79A.1A; no longer IC79A.1B
- net DATA5: now also IC79A.2A; no longer IC79A.2B
- net DATA6: now also IC79A.3A; no longer IC79A.3B
- net DATA7: now also IC79A.4A; no longer IC79A.4B
- net DATA_BUS_ENABLE_LATCH: now also IC34A.O; no longer IC101A.O
- net FILL_LR_H_SAVE_LR: now also IC5D.I0; no longer IC2D.I0
- net FILL_LR_L_SAVE_LR: now also IC5C.I0; no longer IC1B.I0
- net FILL_PC_H_RET: now also IC1B.I0; no longer IC1A.I0
- net FILL_PC_L_JMP_O: now also IC101C.I1; no longer IC101D.I1
- net FILL_PTR_H_SET_PTR: now also IC5A.I1; no longer IC2B.I1
- net FILL_PTR_L_SET_PTR: now also IC169C.I1; no longer IC2A.I1
- net GND: now also IC6A.A, IC6A.B, IC6A.C, IC6A.D, IC7A.A, IC7A.B, IC7A.C, IC7A.D, JP1.11, JP1.13, JP1.7, JP1.9; no longer IC102A.D7, IC105A.D7, IC106A.D7, IC111A.D7, IC113A.D7, IC114A.D7, IC115A.D7, IC98A.D7, JP1.16, JP1.18, JP1.20, JP1.3, JP6.1
- net INPUT_REG0/OPCODE_5/OPCODE_4_IS_NULL: now also IC101A.I0, IC31B.I1; no longer IC34A.I0, IC40B.I1
- net INPUT_REG2: now also IC34B.I0; no longer IC134A.I0, IC134B.I0
- net INPUT_REG3: no longer IC134C.I0, IC134D.I0
- net INPUT_REG_IS_NOT_OUTPUT_REG: now also IC5B.I0; no longer IC43E.I
- net IR_DATA_OUT_7: now also IC101B.I0; no longer IC101C.I0, IC36D.I0, IC49C.I1
- net LR_H_LOAD_INPUT_NOT: now also IC5D.O; no longer IC2D.O
- net LR_H_LOAD_INPUT_TABLE_1: now also IC5D.I1; no longer IC2D.I1
- net LR_L_LOAD_INPUT_NOT: now also IC5C.O; no longer IC1B.O
- net LR_L_LOAD_INPUT_TABLE_1: now also IC5C.I1; no longer IC1B.I1
- net N$11: now also IC169C.O, IC43E.I; no longer IC110B.O, IC52D.I1
- net N$12: now also IC34C.O, IC35E.I; no longer IC40D.O, IC49D.I1
- net N$121: now also IC52D.I0; no longer IC169C.I0
- net N$13: now also IC26D.I0, IC80C.O; no longer IC108A.I0, IC112A.O
- net N$139: now also IC101C.O, IC101D.I1; no longer IC101C.I1, IC101D.O
- net N$141: now also IC49C.O; no longer IC26D.O
- net N$142: now also IC49C.I0; no longer IC26D.I0
- net N$185: now also IC55B.I1; no longer IC108D.I1
- net N$187: now also IC55B.I0; no longer IC108D.I0
- net N$190: now also IC108A.I1, IC108D.O; no longer IC55B.O, IC80C.I1
- net N$192: now also IC108A.I0; no longer IC80C.I0
- net N$193: now also IC108A.O; no longer IC80C.O
- net N$2: now also IC110B.I0; no longer IC52D.I0
- net N$20: now also IC55B.O; no longer IC108D.O
- net N$203: now also IC26D.I1, IC31B.O; no longer IC40B.O, IC80A.I1
- net N$21: now also IC31B.I0, IC80C.I1; no longer IC108A.I1, IC40B.I0
- net N$219: now also IC75C.O; no longer IC31B.O
- net N$22: now also IC101A.O; no longer IC34A.O
- net N$235: no longer IC134B.I1, IC134D.I1
- net N$239: now also IC34B.I1; no longer IC134A.I1, IC134C.I1
- net N$252: now also IC52D.I1; no longer IC169C.I1
- net N$266: now also IC34A.I1, IC34C.I1, IC52D.O; no longer IC101A.I1, IC169C.O, IC40D.I1
- net N$33: now also IC1B.O; no longer IC1A.O
- net N$45: now also IC26D.O, IC5B.I1; no longer IC40C.I1, IC80A.O
- net N$52: now also IC35E.O; no longer IC49D.O
- net N$57: now also IC8B.I1; no longer IC32B.I1
- net N$64: now also IC8C.I1; no longer IC32C.I1
- net N$7: now also IC34A.I0; no longer IC101A.I0
- net N$71: now also IC8D.I1; no longer IC32D.I1
- net N$9: now also IC8A.I1; no longer IC32A.I1
- net N$90: now also IC110B.O; no longer IC52D.O
- net OPCODE_5: no longer IC31B.I1
- net OPC_67_OUPUT0/REG0_JMP: now also IC101A.I1; no longer IC34A.I1
- net PC_COUNT_UP: now also IC1A.O; no longer IC2C.O
- net PC_COUNT_UP_FETCH1: now also IC1A.I0; no longer IC2C.I0
- net PC_COUNT_UP_FETCH2/CYCL_5: now also IC1A.I1; no longer IC2C.I1
- net PC_DATA_OUT_0: now also IC77A.1B; no longer IC77A.1A
- net PC_DATA_OUT_1: now also IC77A.2B; no longer IC77A.2A
- net PC_DATA_OUT_2: now also IC77A.3B; no longer IC77A.3A
- net PC_DATA_OUT_3: now also IC77A.4B; no longer IC77A.4A
- net PC_DATA_OUT_4: now also IC79A.1B; no longer IC79A.1A
- net PC_DATA_OUT_5: now also IC79A.2B; no longer IC79A.2A
- net PC_DATA_OUT_6: now also IC79A.3B; no longer IC79A.3A
- net PC_DATA_OUT_7: now also IC79A.4B; no longer IC79A.4A
- net PC_H_COUNT_DOWN_JMP_O: now also IC101B.O, IC181A.DN; no longer IC101C.O, IC75C.I0
- net PC_H_COUNT_UP_JMP_O: now also IC101D.O, IC49C.I1; no longer IC101B.O, IC26D.I1
- net PC_H_LOAD_INPUT_TABLE_1: now also IC1B.I1; no longer IC1A.I1
- net PTR_H_LOAD_INPUT_NOT: now also IC5A.O; no longer IC2B.O
- net PTR_L_LOAD_INPUT_NOT: now also IC43E.O; no longer IC2A.O
- net REG0_ZERO: now also JP1.20; no longer JP1.11
- net REGISTER_OUTPUT_SEL_3: now also IC34C.I0; no longer IC40D.I0
- net REG_0_LOAD_INPUT: now also IC8A.O; no longer IC32A.O
- net REG_0_OUT_2: now also IC108D.I0; no longer IC55B.I0
- net REG_0_OUT_3: now also IC108D.I1; no longer IC55B.I1
- net REG_1_LOAD_INPUT: now also IC8B.O; no longer IC32B.O
- net REG_2_LOAD_INPUT: now also IC8C.O; no longer IC32C.O
- net REG_3_LOAD_INPUT: now also IC8D.O; no longer IC32D.O
- net SAVE_LR/RET: now also IC75C.I0; no longer IC35E.I
- net SELECT_CARRY_BIT: now also IC34D.I1; no longer IC40A.I1
- net SP_DATA_OVER/UNDERFLOW: now also JP1.18; no longer JP1.9
- net TABLE_1_INPUT_PTR_HIGH: now also IC5A.I0; no longer IC2B.I0
- net TABLE_1_INPUT_PTR_L: now also IC169C.I0; no longer IC2A.I0
- net TABLE_1_INPUT_REG0: now also IC8A.I0; no longer IC32A.I0
- net TABLE_1_INPUT_REG1: now also IC8B.I0; no longer IC32B.I0
- net TABLE_1_INPUT_REG2: now also IC8C.I0; no longer IC32C.I0
- net TABLE_1_INPUT_REG3: now also IC8D.I0; no longer IC32D.I0
- net TWO_BYTE_CMD: now also IC5B.O; no longer IC40C.O
- net VCC: now also IC180A.DN, IC6A.DN, IC6A.LD, IC7A.DN, IC7A.LD; no longer IC49C.I0, IC49D.I0, JP6.2
- net WRITE_REGB_TO_DBUS_JMP_O: no longer IC110B.I0
Other:
- note added: "Timer"
- note added: "unused"
- moved on the sheet: C1, C10, C100, C101, C11, C110, C111, C112, C113, C114, C116, C117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

Commit message: got rid of two cycles! finetuning next
Parts:
- removed C100, C101, C124, C149, C155, C37, C54, C62: (no value), rcl:C-EUC1206
- removed IC117: 74HC74N, 74xx-eu:74HC74N
- removed IC169, IC172, IC190, IC29, IC33: 74HCT32N, 74xx-eu:74HCT32N
- removed IC38, IC75, IC81: 74HCT08N, 74xx-eu:74HCT08N
- removed JP4: (no value), pinhead:PINHD-2X15
- added IC2, IC25: 74HCT32N, 74xx-eu:74HCT32N
Connections:
- removed net CLR_NOT_CS_LDR: IC173A.I0, IC173B.O, IC17B.I0
- removed net CLR_NOT_CS_POP: IC172C.O, IC48D.I0, IC85C.I1
- removed net CONNECT_REG_TO_DBUS_PTR: IC172D.O, IC52B.I0
- removed net FILL_LR_H_SAVE_LR: IC29C.I0, IC5D.I0, IC81A.O
- removed net FILL_LR_L_SAVE_LR: IC29A.I0, IC5C.I0, IC81C.O
- removed net FILL_PC_H_RET: IC1B.I0, IC29D.I0, IC51D.O
- removed net FILL_PC_L_JMP_O: IC101C.I1, IC1D.I0, IC33A.I0, IC38D.O
- removed net FILL_PC_L_RET: IC1D.I1, IC29B.I0, IC51A.O
- removed net FILL_PTR_H_SET_PTR: IC169A.I0, IC26C.O, IC5A.I1
- removed net FILL_PTR_L_PTR_ADD: IC24C.O, IC31D.I1, IC33A.I1
- removed net FILL_PTR_L_SET_PTR: IC169C.I1, IC172D.I0, IC26A.O
- removed net FILL_REGISTER_ALU/ALU_TO_DBUS: IC117B.CLK, IC169B.I0, IC169D.I1, IC75D.O
- removed net FILL_REGISTER_LDR: IC108B.I1, IC173B.I0, IC27B.O
- removed net FILL_REGISTER_MOV: IC169D.I0, IC190B.I0, IC74B.O
- removed net FILL_REGISTER_POP: IC108B.I0, IC172C.I0, IC24B.O
- removed net IR_LOAD_INPUT: IC127A.O, IC80D.I0, IC90A.CLK
- removed net N$112: IC29A.I1, IC81D.O
- removed net N$122: IC173B.I1, IC27A.O
- removed net N$143: IC168B.I0, IC168D.O
- removed net N$147: IC169B.I1, IC33A.O
- removed net N$155: IC168A.O, IC168D.I0
- removed net N$156: IC172C.I1, IC24A.O
- removed net N$160: IC169A.I1, IC26B.O
- removed net N$18: IC169B.O, IC43D.I
- removed net N$196: IC172D.I1, IC24D.O
- removed net N$204: IC190A.I1, IC74C.O
- removed net N$223: IC29B.I1, IC51B.O
- removed net N$226: IC29D.I1, IC51C.O
- removed net N$233: IC29C.I1, IC81B.O
- removed net N$56: IC190B.I1, IC74A.O
- removed net PC_COUNT_UP_FETCH2/CYCL_5: IC14A.Q, IC14B.D, IC1A.I1, JP1.30
- removed net PC_HIGH_LOAD_INPUT_JMP: IC190C.I0, IC28D.O, IC48B.I0
- removed net PC_LOW_LOAD_INPUT_JMP: IC190A.I0, IC1C.I0, IC74D.O
- removed net STATE_0/CYCL_6: IC125A.I0, IC14B.Q, IC15A.D, IC23D.I0, IC24D.I0, IC27C.I0, IC28A.I0, IC31C.I0, IC38C.I0, IC51B.I0, IC74A.I0, IC74C.I0, IC78D.I0, IC81D.I0, JP1.32
- removed net STATE_1/CYCL_7: IC15A.Q, IC15B.D, IC23A.I0, IC23B.I0, IC24A.I0, IC26A.I0, IC27A.I0, IC27D.I0, IC38A.I0, IC51A.I0, IC74B.I0, IC74D.I0, IC75A.I0, IC81C.I0, JP1.34
- removed net STATE_2/CYCL_8: IC117A.D, IC15B.Q, IC23C.I0, IC24B.I0, IC26B.I0, IC27B.I0, IC28B.I0, IC28C.I0, IC38B.I0, IC51C.I0, IC75B.I0, IC81B.I0, JP1.36
- removed net STATE_3/CYCL_9: IC10A.D, IC117A.Q, IC24C.I0, IC26C.I0, IC28D.I0, IC31A.I0, IC38D.I0, IC51D.I0, IC75D.I0, IC81A.I0, JP1.38
- removed net WRITE_LR_H_DBUS_RET: IC141A.I1, IC29D.O, IC36B.I0
- removed net WRITE_LR_L_DBUS_RET: IC141A.I0, IC29B.O
- removed net WRITE_PC_H_DBUS_SAVE_LR: IC141D.I1, IC29C.O
- removed net WRITE_PC_L_DBUS_SAVE_LR: IC141D.I0, IC29A.O, IC36B.I1
- removed net WRITE_REGB_TO_DBUS_ALU: IC168C.I0, IC75B.O
- removed net WRITE_REGB_TO_DBUS_JMP: IC168D.I1, IC190C.O
- removed net WRITE_REGB_TO_DBUS_JMP_O: IC168A.I1, IC38B.O
- removed net WRITE_REGB_TO_DBUS_PTR_ADD: IC168A.I0, IC28B.O
- removed net WRITE_REGB_TO_DBUS_SET_PTR: IC168C.I1, IC169A.O
- removed net WRITE_REG_TO_DBUS_JMP: IC190A.O, IC52A.I0
- removed net WRITE_REG_TO_DBUS_MOV: IC190B.O, IC52B.I1
- new net CLR_NOT_CS_LDR/FILL_REGISTER_LDR: IC108B.I1, IC173A.I0, IC17B.I0, IC27C.O
- new net CLR_NOT_CS_POP/FILL_REGISTER_POP: IC108B.I0, IC125A.O, IC48D.I0, IC85C.I1
- new net CONNECT_REG_TO_DBUS_PTR/FILL_PTR_L_SET_PTR: IC24D.O, IC48A.I1, IC52B.I0
- new net IR_LOAD_INPUT/PC_COUNT_UP_FETCH2: IC127A.O, IC1A.I1, IC80D.I0, IC90A.CLK
- new net PTR_ADD_OR_JMP_O_OR_ALU_FILL: IC168B.I0, IC168C.O, IC43D.I
- new net STATE_0/CYCL_5: IC14A.Q, IC14B.D, IC24A.I0, IC24B.I0, IC24C.I0, IC24D.I0, IC31C.I0, IC51B.I0, IC51C.I0, IC51D.I0, IC74A.I0, IC74B.I0, IC74C.I0, IC74D.I0, JP1.30
- new net STATE_1/CYCL_6: IC125A.I0, IC14B.Q, IC15A.D, IC23A.I0, IC26A.I0, IC26B.I0, IC27B.I0, IC27C.I0, IC27D.I0, IC28A.I0, IC28C.I0, IC51A.I0, IC78D.I0, JP1.32
- new net STATE_2/CYCL_7: IC10A.D, IC15A.Q, IC23B.I0, IC27A.I0, IC28B.I0, IC28D.I0, IC31A.I0, JP1.34
- new net WRITE_LR_H_DBUS_RET/FILL_PC_H_RET: IC141A.I1, IC1B.I0, IC36B.I0, IC51A.O
- new net WRITE_LR_L_DBUS_RET/FILL_PC_L_RET: IC141A.I0, IC1D.I1, IC24A.O
- new net WRITE_PC_H_DBUS_SAVE_LR/FILL_LR_H_SAVE_LR: IC141D.I1, IC26B.O, IC5D.I0
- new net WRITE_PC_L_DBUS_SAVE_LR/FILL_LR_L_SAVE_LR: IC141D.I0, IC24C.O, IC36B.I1, IC5C.I0
- new net WRITE_REGB_TO_DBUS_ALU/FILL_REGISTER_ALU/ALU_TO_DBUS: IC15B.CLK, IC168C.I1, IC23B.O, IC2D.I1
- new net WRITE_REGB_TO_DBUS_JMP/PC_HIGH_LOAD_INPUT_JMP: IC168D.I0, IC28C.O, IC5B.I0
- new net WRITE_REGB_TO_DBUS_JMP_O/FILL_PC_L_JMP_O: IC101C.I1, IC168A.I1, IC1D.I0, IC28D.O
- new net WRITE_REGB_TO_DBUS_PTR_ADD/FILL_PTR_L_PTR_ADD: IC168A.I0, IC28B.O, IC31D.I1
- new net WRITE_REGB_TO_DBUS_SET_PTR/FILL_PTR_H_SET_PTR: IC168D.I1, IC26A.O, IC48B.I1
- new net WRITE_REG_TO_DBUS_JMP/PC_LOW_LOAD_INPUT_JMP: IC1C.I0, IC52A.I0, IC74C.O
- new net WRITE_REG_TO_DBUS_MOV/FILL_REGISTER_MOV: IC2D.I0, IC52B.I1, IC74A.O
- net !CLR_CARRY_BIT: now also IC15B.CLR; no longer IC117B.CLR
- net !OPCODE_5: now also IC26C.I1; no longer IC75C.I1
- net !RING_CNTR_RESET: no longer IC117A.CLR, IC15B.CLR
- net !SET_CARRY_BIT: now also IC15B.PRE; no longer IC117B.PRE
- net ADRR_0: no longer JP3.1
- net ADRR_1: no longer JP3.3
- net ADRR_10: no longer JP3.21
- net ADRR_11: no longer JP3.23
- net ADRR_12: no longer JP3.25
- net ADRR_13: no longer JP3.27
- net ADRR_14: no longer JP3.29
- net ADRR_2: no longer JP3.5
- net ADRR_3: no longer JP3.7
- net ADRR_4: no longer JP3.9
- net ADRR_5: no longer JP3.11
- net ADRR_6: no longer JP3.13
- net ADRR_7: no longer JP3.15
- net ADRR_8: no longer JP3.17
- net ADRR_9: no longer JP3.19
- net ALU_CARRY_BIT: now also IC15B.Q; no longer IC117B.Q
- net ALU_CARRY_OUT: now also IC15B.D; no longer IC117B.D
- net ALU_NR1_ENABLE_ALU: now also IC25C.I0; no longer IC33C.I0
- net ALU_NR1_ENABLE_JMP_O_PTR_ADD: now also IC25C.I1; no longer IC33C.I1
- net ALU_NR2_ENABLE_ALU: now also IC25D.I0; no longer IC33B.I0
- net ALU_NR2_ENABLE_JMP_O_PTR_ADD: now also IC25D.I1; no longer IC33B.I1
- net CLR_NOT_CS_PUSH: now also IC173B.I0, IC27A.O; no longer IC172A.I0, IC23C.O
- net CLR_NOT_OE/CLR_NOT_CS_CYCL_0: now also IC85D.I0; no longer IC48C.I0
- net CLR_NOT_OE_POP: now also JP3.4; no longer JP4.20
- net CONNECT_PTR_TO_ABUS/CLR_NOT_OE_LDR: now also IC85D.I1; no longer IC48C.I1
- net CONNECT_PTR_TO_ABUS/CONNECT_REG_TO_DBUS/CLR_NOT_WE/SELECTOR_TABLE_2_STR: now also IC2C.I0; no longer IC124A.I0
- net CONNECT_REG_TO_DBUS/CLR_NOT_WE/SELECTOR_TABLE_2_PUSH: now also IC173B.O, IC2C.I1; no longer IC124A.I1, IC172A.O
- net DATA0: no longer JP3.2, JP4.2
- net DATA1: no longer JP3.4, JP4.4
- net DATA2: no longer JP3.6, JP4.6
- net DATA3: no longer JP3.8, JP4.8
- net DATA4: no longer JP3.10, JP4.10
- net DATA5: no longer JP3.12, JP4.12
- net DATA6: no longer JP3.14, JP4.14
- net DATA7: no longer JP3.16, JP4.16
- net DBUS_SELECTOR_TABLE_2: now also IC2C.O; no longer IC124A.O
- net GND: now also JP1.36, JP1.38, JP3.10, JP3.14, JP3.2; no longer C100.2, C101.2, C124.2, C149.2, C155.2, C37.2, C54.2, C62.2, JP4.18, JP4.26, JP4.30
- net HGGJHGGJZGZ77UZGHGHHGHGHGHGHJGHJ: now also IC51C.O; no longer IC28A.O
- net INPUT_REG_IS_NOT_OUTPUT_REG: now also IC108C.I0, IC2B.O; no longer IC108C.O, IC5B.I0
- net LATCH_ALU_INPUT_B_ALU: now also IC124A.I0, IC28A.O; no longer IC190D.I0, IC75A.O
- net LATCH_ALU_INPUT_B_JMP_O: now also IC78D.O, IC80A.I0; no longer IC172B.I0, IC38A.O
- net LDR: now also IC27C.I1, IC51C.I1; no longer IC27A.I1, IC27B.I1, IC28A.I1
- net MEM_NOT_OE: now also IC85D.O; no longer IC48C.O
- net N$109: now also IC74D.O, IC80A.I1; no longer IC172B.I1, IC38C.O
- net N$11: now also IC168A.O, IC168C.I0; no longer IC169C.O, IC43E.I
- net N$110: now also IC124A.I1, IC74B.O; no longer IC190D.I1, IC78D.O
- net N$123: now also IC51D.O; no longer IC27C.O
- net N$132: now also IC28D.I1, IC74D.I1, IC78D.I1; no longer IC38A.I1, IC38B.I1, IC38C.I1, IC38D.I1
- net N$146: now also IC173B.I1, IC27B.O; no longer IC172A.I1, IC23B.O
- net N$148: now also IC25D.O; no longer IC33B.O
- net N$15: no longer IC28D.I1, IC74D.I1
- net N$151: now also IC24B.O; no longer IC125A.O
- net N$157: now also IC51B.O; no longer IC23D.O
- net N$163: now also IC5A.I1; no longer IC48A.I1
- net N$193: now also IC48C.I0; no longer IC85D.I0
- net N$194: now also IC24C.I1, IC26B.I1; no longer IC81A.I1, IC81B.I1, IC81C.I1, IC81D.I1
- net N$20: now also IC48C.I1; no longer IC85D.I1
- net N$202: now also IC25C.O; no longer IC33C.O
- net N$219: now also IC24A.I1, IC26C.O; no longer IC51B.I1, IC51C.I1, IC51D.I1, IC75C.O
- net N$236: now also JP3.8; no longer JP4.24
- net N$237: now also JP3.6; no longer JP4.22
- net N$32: now also IC5A.I0; no longer IC48A.I0
- net N$33: now also IC5B.I1; no longer IC48B.I1
- net N$4: now also IC168D.O; no longer IC168C.O
- net N$45: now also IC108C.I1; no longer IC5B.I1
- net N$47: now also IC2A.O; no longer IC33D.O
- net N$48: now also IC2B.I0; no longer IC108C.I0
- net N$5: now also IC108C.O, IC43E.I; no longer IC190C.I1, IC28C.O
- net N$51: now also IC2B.I1; no longer IC108C.I1
- net N$55: no longer IC74B.I1
- net N$6: now also IC2D.O; no longer IC169D.O
- net N$97: no longer IC26B.I1, IC26C.I1
- net PC_HIGH_LOAD_INPUT_NOT: now also IC5B.O; no longer IC48B.O
- net PC_LOW_LOAD_INPUT_NOT: now also IC5A.O; no longer IC48A.O
- net POP: now also IC125A.I1, IC51B.I1; no longer IC23D.I1, IC24A.I1, IC24B.I1
- net PTR_ADD: now also IC24B.I1; no longer IC125A.I1, IC24C.I1
- net PTR_H_LOAD_INPUT_NOT: now also IC48B.O; no longer IC5A.O
- net PTR_L_LOAD_INPUT_NOT: now also IC48A.O; no longer IC43E.O
- net PUSH: now also IC27A.I1, IC27B.I1; no longer IC23B.I1, IC23C.I1
- net REG0_ZERO: now also IC48C.O; no longer IC85D.O
- net RING_CNTR_CLOCK: no longer IC117A.CLK, IC15B.CLK
- net SAVE_LR/RET: now also IC26C.I0; no longer IC75C.I0
- net SECOND_LATCH_SELECT: now also IC2A.I0; no longer IC33D.I0
- net SELECT_CARRY_BIT: now also IC23B.I1, IC28A.I1, IC74B.I1; no longer IC75A.I1, IC75B.I1, IC75D.I1, IC78D.I1
- net SP_DATA_OUT_0: now also JP3.1; no longer JP4.1
- net SP_DATA_OUT_1: now also JP3.3; no longer JP4.3
- net SP_DATA_OUT_10: now also JP3.21; no longer JP4.21
- net SP_DATA_OUT_11: now also JP3.23; no longer JP4.23
- net SP_DATA_OUT_12: now also JP3.25; no longer JP4.25
- net SP_DATA_OUT_13: now also JP3.27; no longer JP4.27
- net SP_DATA_OUT_14: now also JP3.29; no longer JP4.29
- net SP_DATA_OUT_2: now also JP3.5; no longer JP4.5
- net SP_DATA_OUT_3: now also JP3.7; no longer JP4.7
- net SP_DATA_OUT_4: now also JP3.9; no longer JP4.9
- net SP_DATA_OUT_5: now also JP3.11; no longer JP4.11
- net SP_DATA_OUT_6: now also JP3.13; no longer JP4.13
- net SP_DATA_OUT_7: now also JP3.15; no longer JP4.15
- net SP_DATA_OUT_8: now also JP3.17; no longer JP4.17
- net SP_DATA_OUT_9: now also JP3.19; no longer JP4.19
- net STR: now also IC51D.I1; no longer IC27C.I1
- net TABLE_1_INPUT_PTR_HIGH: now also IC48B.I0; no longer IC5A.I0
- net TABLE_1_INPUT_PTR_L: now also IC48A.I0; no longer IC169C.I0
- net TWO_BYTE_CMD: now also IC43E.O; no longer IC5B.O
- net VCC: now also JP3.12; no longer C100.1, C101.1, C124.1, C149.1, C155.1, C37.1, C54.1, C62.1, IC117A.PRE, IC15B.PRE, JP4.28
- net WRITE_PC_L_ALU_LATCH_JMP_O: now also IC80A.O; no longer IC172B.O
- net WRITE_PTR_L_TO_DBUS_PTR_ADD: now also IC2A.I1; no longer IC33D.I1
- net WRITE_REG_TO_DBUS_ALU: now also IC124A.O; no longer IC190D.O
Other:
- note added: "Do we need a pause between both CS/Read Cycles?"
- note removed: "CYCL_8"
- note removed: "CYCL_9"
- moved on the sheet: C14, C20, C21, C22, C23, C26, C27, C29, C30, C31, C32, C33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

Commit message: clean up docs and schematic. no functional changes
Connections:
- net CONNECT_PTR_TO_ABUS/CONNECT_REG_TO_DBUS/CLR_NOT_WE/SELECTOR_TABLE_2_STR renamed CNNCT_PTR_TO_ABUS/CNNCT_REG_TO_DBUS/CLR_NOT_WE/SELECTOR_2_STR
- net INPUT_REG0/OPCODE_5/OPCODE_4_IS_NULL renamed INPUT_REG0/OPC4/5_IS_NULL
- net UNUSED renamed NOT_USED1
Other:
- moved on the sheet: IC17C, IC17D, IC2C, IC35B, IC35E, IC36B, IC46, IC85D, IC8A, IC8B, IC8C, IC8D

Commit message: fix ui_bord. seems to work
Other:
- moved on the sheet: IC124C, IC124D, IC125D, IC28C, IC36B, IC74C, IC78C
