File: schematics/Control_Unit/Control_Unit.sch (EAGLE design)
At the start: 222 parts, among them IC1 74HCT32N, IC10 74HC74N, IC100 74HCT374N, IC101 74HCT08N, IC102 74HC151N, IC103 74HC373N, IC105 74HC151N, IC106 74HC151N, IC108 74HCT32N, IC11 74HC74N, IC110 74HCT32N, IC111 74HC151N, IC112 74HCT32N, IC113 74HC151N, IC114 74HC151N, IC115 74HC151N, IC116 74HC373N, IC12 74AC08N, IC124 74HCT32N, IC125 74HCT08N, IC126 74AC157N, IC127 74HCT08N, IC128 74AC08N, IC129 74AC08N, IC13 74AC08N, IC135 74HCT08N, IC136 74HCT08N, IC14 74HC74N, IC141 74HCT32N, IC15 74HC74N, IC16 74AC08N, IC168 74HCT32N, IC17 74HCT32N, IC173 74HCT32N, IC175 74HC193N, IC176 74HC193N, IC177 74HC193N, IC178 74HC193N, IC179 74HC193N, IC18 74AC08N, IC180 74HC193N, IC181 74HC193N, IC182 74HC193N, IC19 74AC08N, IC191 74HCT32N, IC2 74HCT32N, IC20 74AC08N, IC21 74AC08N, IC22 74HCT32N, IC23 74HCT08N, IC24 74HCT08N, IC25 74HCT32N, IC26 74HCT08N, IC27 74HCT08N, IC28 74HCT08N, IC3 74HC151N, IC30 74HCT08N, IC31 74HCT00N, IC34 74HCT08N, IC35 74HCT04N, IC36 74HCT32N, IC39 74HCT08N, IC4 74AC08N, IC41 74HCT08N, IC42 74HC373N, IC43 74HCT04N, IC44 74ACT157N, IC46 74ACT157N, IC47 74HCT04N, IC48 74ACT02N, IC49 74AC86N, IC5 74ACT02N, IC51 74HCT08N, IC52 74HCT32N, IC55 74HCT32N, IC56 74HC151N, IC57 74HC151N, IC58 74HC151N, IC59 74HC151N, IC6 74HC193N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

Commit message: finished COntrolUnit. Not much left to do
Connections:
- net CNNCT_PTR_TO_ABUS/CNNCT_REG_TO_DBUS/CLR_NOT_WE/SELECTOR_2_STR renamed CNNCT_PTR_TO_ABUS/CNNCT_REG_TO_DBUS/CLR_NOT_WE/SEL_2_STR
- net WRITE_LR_H_DBUS_RET/FILL_PC_H_RET renamed WRITE_LR_H_DBUS/FILL_PC_H_RET
- net WRITE_PC_L_DBUS_SAVE_LR/FILL_LR_L_SAVE_LR renamed WRITE_PC_L_DBUS/FILL_LR_L_SAVE_LR
- net WRITE_REGB_TO_DBUS_ALU/FILL_REGISTER_ALU/ALU_TO_DBUS renamed WRITE_REGB_TO_DBUS/FILL_REGISTER/ALU_TO_DBUS_ALU
- net WRITE_REGB_TO_DBUS_JMP_O/FILL_PC_L_JMP_O renamed WRITE_REGB_TO_DBUS/FILL_PC_L_JMP_O
- net WRITE_REGB_TO_DBUS_PTR_ADD/FILL_PTR_L_PTR_ADD renamed WRITE_REGB_TO_DBUS/FILL_PTR_L_PTR_ADD
- removed net CYCL_3: IC11A.Q, IC11B.D, IC127D.I1, JP1.26
- removed net CYCL_4: IC11B.Q, IC127A.I0, IC14A.D, JP1.28
- removed net IR_LOAD_INPUT/PC_COUNT_UP_FETCH2: IC127A.O, IC1A.I1, IC80D.I0, IC90A.CLK
- removed net NOT_USED1: IC34B.O
- removed net PC_COUNT_UP_FETCH1: IC127D.O, IC1A.I0, IC80D.I1
- new net !TWO_BYTE_CMD: IC108C.O, IC23C.I1, IC43E.I
- new net IR_LOAD_INPUT/PC_COUNT_UP_FETCH2/CYCL_4: IC11B.Q, IC1A.I1, IC25A.I0, IC80D.I0, IC90A.CLK, JP1.28
- new net N$44: IC11A.Q, IC23C.I0, IC23D.I0
- new net N$56: IC14A.D, IC25A.O
- new net PC_COUNT_UP_FETCH1/CYCL_3: IC11B.D, IC1A.I0, IC23D.O, IC80D.I1, JP1.26
- net !IR_DATA_OUT_7: now also IC127C.I1; no longer IC127C.I0
- net ALU_CARRY_BIT: now also IC34B.I0; no longer IC34D.I0
- net ALU_CARRY_IN: now also IC34B.O; no longer IC34D.O
- net DATA_BUS_ENABLE_LATCH: now also IC127A.O; no longer IC34A.O
- net GND: now also JP9.36, JP9.38
- net INPUT_REG2: no longer IC34B.I0
- net N$12: now also IC127D.O; no longer IC34C.O
- net N$132: now also IC124B.I0; no longer IC124B.I1
- net N$166: now also IC127C.I0; no longer IC127C.I1
- net N$239: no longer IC34B.I1
- net N$266: now also IC127A.I1, IC127D.I1; no longer IC34A.I1, IC34C.I1
- net N$5: now also IC23C.O, IC25A.I1; no longer IC108C.O, IC43E.I
- net N$7: now also IC127A.I0; no longer IC34A.I0
- net PC_L_LOAD_INPUT_TABLE_1: now also IC1D.I1; no longer IC1C.I1
- net PTR_ADD: now also IC124B.I1; no longer IC124B.I0
- net REGISTER_OUTPUT_SEL_3: now also IC127D.I0; no longer IC34C.I0
- net SELECT_CARRY_BIT: now also IC34B.I1; no longer IC34D.I1
- net TWO_BYTE_CMD: now also IC23D.I1; no longer IC127A.I1, IC127D.I0
- net WRITE_LR_L_DBUS_RET/FILL_PC_L_RET: now also IC1C.I1; no longer IC1D.I1
Other:
- note added: "CYCL_3"
- note added: "CYCL_4"
- note added: "Maybe we can omit the first FF and do the SIgnal int Cycl7"
- note added: "PC only counts up"
- note removed: "PC only counts up. Put Count down on HIGH"
- note removed: "unused"
- moved on the sheet: IC108C, IC10A, IC10B, IC112A, IC112B, IC112C, IC112D, IC11A, IC124B, IC125C, IC127A, IC127C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

Commit message: improve layout
Connections:
- net CLR_NOT_CS_LDR/FILL_REGISTER_LDR renamed CLR_NOT_CS/FILL_REGISTER_LDR
- net WRITE_PC_H_DBUS_SAVE_LR/FILL_LR_H_SAVE_LR renamed WRITE_PC_H_DBUS/FILL_LR_H_SAVE_LR
- net WRITE_REGB_TO_DBUS_SET_PTR/FILL_PTR_H_SET_PTR renamed WRITE_REGB_TO_DBUS/FILL_PTR_H_SET_PTR
Other:
- note added: "Addr15 decides whether to use RAM or FLASH"
- note added: "I am not happy with the memory. Too much FLash and too little RAM"
- note added: "Operand byte storage for two-byte instructions"
- note removed: "Addr15 goes to Enable of the mem chips"
- note removed: "Here is the operand byte stored for two-byte instructions"
- moved on the sheet: IC103, IC108A, IC108D, IC110C, IC110D, IC15B, IC17A, IC17B, IC17C, IC17D, IC25C, IC25D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

Commit message: fix latex docs
Connections:
- net CLR_NOT_OE/CLR_NOT_CS_CYCL_0 renamed CLR_NOT_OE/CLR_NOT_CS_CYCL_1/2
- net CLR_NOT_OE/CLR_NOT_CS_CYCL_2 renamed CLR_NOT_OE/CLR_NOT_CS_CYCL_3/4
- net WRITE_REGB_TO_DBUS_JMP/PC_HIGH_LOAD_INPUT_JMP renamed WRITE_REGB_TO_DBUS/PC_HIGH_LOAD_INPUT_JMP
Other:
- moved on the sheet: IC100, IC173C, IC42, IC43D

Commit message: renumber schematic parts
Parts:
- removed C117, C120, C121, C122, C123, C127, C142, C143, C145, C148, C150, C151, C154: (no value), rcl:C-EUC1206
- removed IC110, IC112, IC124, IC168, IC173, IC191: 74HCT32N, 74xx-eu:74HCT32N
- removed IC113, IC114, IC115: 74HC151N, 74xx-eu:74HC151N
- removed IC116: 74HC373N, 74xx-eu:74HC373N
- removed IC125, IC127, IC135, IC136: 74HCT08N, 74xx-eu:74HCT08N
- removed IC126: 74AC157N, 74xx-eu:74AC157N
- removed IC128, IC129: 74AC08N, 74xx-eu:74AC08N
- removed IC175, IC176, IC177, IC179, IC180, IC181, IC182: 74HC193N, custom_parts:74HC193N
- removed JP10: (no value), pinhead:PINHD-2X20
- added C108, C24, C25, C37, C41, C45, C46, C54, C62, C66, C69, C76, C81: (no value), rcl:C-EUC1206
- added IC104: 74ACT157N, 74xx-eu:74ACT157N
- added IC107, IC62, IC76, IC92: 74HCT08N, 74xx-eu:74HCT08N
- added IC109: 74HCT00N, 74xx-eu:74HCT00N
- added IC29: 74ACT02N, 74xx-eu:74ACT02N
- added IC33, IC45, IC66, IC81: 74HCT374N, 74xx-eu:74HCT374N
- added IC37, IC38, IC50: 74HC151N, 74xx-eu:74HC151N
- added IC40, IC68, IC94, IC96: 74HCT32N, 74xx-eu:74HCT32N
- added IC53, IC54: 74HC74N, 74xx-eu:74HC74N
- added IC67: 74HCT04N, 74xx-eu:74HCT04N
- added IC69, IC75: 74HC193N, custom_parts:74HC193N
- added IC95: 74AC08N, 74xx-eu:74AC08N
- added JP4: (no value), pinhead:PINHD-2X20
- IC10: value 74HC74N -> 74HCT08N; device 74xx-eu:74HC74N -> 74xx-eu:74HCT08N
- IC100, IC99: value 74HCT374N -> 74HCT08N; device 74xx-eu:74HCT374N -> 74xx-eu:74HCT08N
- IC101: value 74HCT08N -> 74HC373N; device 74xx-eu:74HCT08N -> 74xx-eu:74HC373N
- IC102, IC106, IC57, IC58, IC60: value 74HC151N -> 74HC193N; device 74xx-eu:74HC151N -> custom_parts:74HC193N
- IC105, IC56, IC61: value 74HC151N -> 74HCT32N; device 74xx-eu:74HC151N -> 74xx-eu:74HCT32N
- IC108, IC2: value 74HCT32N -> 74HCT08N; device 74xx-eu:74HCT32N -> 74xx-eu:74HCT08N
- IC11: value 74HC74N -> 74ACT157N; device 74xx-eu:74HC74N -> 74xx-eu:74ACT157N
- IC12, IC13, IC21: value 74AC08N -> 74ACT157N; device 74xx-eu:74AC08N -> 74xx-eu:74ACT157N
- IC14: value 74HC74N -> 74HCT04N; device 74xx-eu:74HC74N -> 74xx-eu:74HCT04N
- IC15: value 74HC74N -> 74HC151N; device 74xx-eu:74HC74N -> 74xx-eu:74HC151N
- IC16, IC4: value 74AC08N -> 74HC151N; device 74xx-eu:74AC08N -> 74xx-eu:74HC151N
- IC18: value 74AC08N -> 74HCT374N; device 74xx-eu:74AC08N -> 74xx-eu:74HCT374N
- IC19: value 74AC08N -> 74ACT02N; device 74xx-eu:74AC08N -> 74xx-eu:74ACT02N
- IC20: value 74AC08N -> 74HCT08N; device 74xx-eu:74AC08N -> 74xx-eu:74HCT08N
- IC22: value 74HCT32N -> 74HC151N; device 74xx-eu:74HCT32N -> 74xx-eu:74HC151N
- IC23, IC51: value 74HCT08N -> 74HC151N; device 74xx-eu:74HCT08N -> 74xx-eu:74HC151N
- IC25: value 74HCT32N -> 74AC86N; device 74xx-eu:74HCT32N -> 74xx-eu:74AC86N
- IC26, IC41: value 74HCT08N -> 74HCT374N; device 74xx-eu:74HCT08N -> 74xx-eu:74HCT374N
- IC27, IC34: value 74HCT08N -> 74ACT157N; device 74xx-eu:74HCT08N -> 74xx-eu:74ACT157N
- IC28: value 74HCT08N -> 74AC08N; device 74xx-eu:74HCT08N -> 74xx-eu:74AC08N
- IC31: value 74HCT00N -> 74HC151N; device 74xx-eu:74HCT00N -> 74xx-eu:74HC151N
- IC35: value 74HCT04N -> 74HC373N; device 74xx-eu:74HCT04N -> 74xx-eu:74HC373N
- IC36: value 74HCT32N -> 74HC373N; device 74xx-eu:74HCT32N -> 74xx-eu:74HC373N
- IC39: value 74HCT08N -> 74ACT02N; device 74xx-eu:74HCT08N -> 74xx-eu:74ACT02N
- IC42: value 74HC373N -> 74HC151N; device 74xx-eu:74HC373N -> 74xx-eu:74HC151N
- IC43, IC47: value 74HCT04N -> 74HC151N; device 74xx-eu:74HCT04N -> 74xx-eu:74HC151N
- IC44: value 74ACT157N -> 74ACT02N; device 74xx-eu:74ACT157N -> 74xx-eu:74ACT02N
- IC46: value 74ACT157N -> 74HC151N; device 74xx-eu:74ACT157N -> 74xx-eu:74HC151N
- IC48, IC8: value 74ACT02N -> 74HCT32N; device 74xx-eu:74ACT02N -> 74xx-eu:74HCT32N
- IC49: value 74AC86N -> 74HCT32N; device 74xx-eu:74AC86N -> 74xx-eu:74HCT32N
- IC5, IC85: value 74ACT02N -> 74HCT374N; device 74xx-eu:74ACT02N -> 74xx-eu:74HCT374N
- IC52, IC55: value 74HCT32N -> 74HC74N; device 74xx-eu:74HCT32N -> 74xx-eu:74HC74N
- IC59: value 74HC151N -> 74HCT08N; device 74xx-eu:74HC151N -> 74xx-eu:74HCT08N
- IC6, IC7, IC82, IC83: value 74HC193N -> 74AC08N; device custom_parts:74HC193N -> 74xx-eu:74AC08N
- IC63, IC70, IC71, IC84: value 74HCT374N -> 74HCT32N; device 74xx-eu:74HCT374N -> 74xx-eu:74HCT32N
- IC64, IC93: value 74HCT374N -> 74HC193N; device 74xx-eu:74HCT374N -> custom_parts:74HC193N
- IC72: value 74HC373N -> 74HCT08N; device 74xx-eu:74HC373N -> 74xx-eu:74HCT08N
- IC74: value 74HCT08N -> 74HC193N; device 74xx-eu:74HCT08N -> custom_parts:74HC193N
- IC77, IC87: value 74ACT157N -> 74AC08N; device 74xx-eu:74ACT157N -> 74xx-eu:74AC08N
- IC79: value 74ACT157N -> 74HCT374N; device 74xx-eu:74ACT157N -> 74xx-eu:74HCT374N
- IC80: value 74HCT32N -> 74HC193N; device 74xx-eu:74HCT32N -> custom_parts:74HC193N
- IC86: value 74ACT157N -> 74HCT04N; device 74xx-eu:74ACT157N -> 74xx-eu:74HCT04N
- IC88, IC89: value 74ACT157N -> 74HCT08N; device 74xx-eu:74ACT157N -> 74xx-eu:74HCT08N
- IC9: value 74HC151N -> 74AC157N; device 74xx-eu:74HC151N -> 74xx-eu:74AC157N
- IC90, IC91: value 74HCT374N -> 74AC08N; device 74xx-eu:74HCT374N -> 74xx-eu:74AC08N
- IC98: value 74HC151N -> 74ACT157N; device 74xx-eu:74HC151N -> 74xx-eu:74ACT157N
- JP1: device pinhead:PINHD-2X20 -> pinhead:PINHD-2X15
- JP3: device pinhead:PINHD-2X15 -> pinhead:PINHD-2X20
- renumbered C110 to C107, C111 to C106, C112 to C103, C113 to C105, C114 to C104, C116 to C102, C118 to C101, C126 to C98, C129 to C100, C130 to C95, C131 to C97, C132 to C96, C141 to C94, C144 to C92, C146 to C89, C147 to C88, C153 to C83, IC111 to IC32, IC141 to IC65, IC178 to IC97, JP9 to JP5
Connections:
- net !CLR_CARRY_BIT: now also IC55B.CLR, JP4.12; no longer IC15B.CLR, JP1.12
- net !IR_DATA_OUT_7: now also IC40D.I0, IC59C.I1, IC86E.O, IC88D.I0; no longer IC101D.I0, IC127C.I1, IC36D.I0, IC47E.O
- net !OPCODE_5: now also IC14C.O, IC28A.I1, IC28B.I1, IC92C.I1; no longer IC129A.I1, IC129B.I1, IC26C.I1, IC43C.O
- net !REGISTER_RESET: now also IC102A.CLR, IC106A.CLR, IC57A.CLR, IC58A.CLR, IC60A.CLR, IC64A.CLR, IC69A.CLR, IC74A.CLR, IC75A.CLR, IC80A.CLR, IC93A.CLR, JP4.8; no longer IC175A.CLR, IC176A.CLR, IC177A.CLR, IC179A.CLR, IC180A.CLR, IC181A.CLR, IC182A.CLR, IC6A.CLR, IC7A.CLR, IC82A.CLR, IC83A.CLR, JP1.8
- net !RING_CNTR_RESET: now also IC52A.PRE, IC52B.CLR, IC53A.CLR, IC53B.CLR, IC54A.CLR, IC54B.CLR, IC55A.CLR, JP4.10; no longer IC10A.PRE, IC10B.CLR, IC11A.CLR, IC11B.CLR, IC14A.CLR, IC14B.CLR, IC15A.CLR, JP1.10
- net !SET_CARRY_BIT: now also IC55B.PRE, JP4.14; no longer IC15B.PRE, JP1.14
- net !TWO_BYTE_CMD: now also IC14E.I, IC89C.I1, IC96C.O; no longer IC108C.O, IC23C.I1, IC43E.I
- net ADRR_0: now also IC13A.1Y, JP1.1; no longer IC86A.1Y, JP2.1
- net ADRR_1: now also IC13A.2Y, JP1.3; no longer IC86A.2Y, JP2.3
- net ADRR_10: now also IC27A.3Y, JP1.21; no longer IC88A.3Y, JP2.21
- net ADRR_11: now also IC27A.4Y, JP1.23; no longer IC88A.4Y, JP2.23
- net ADRR_12: now also IC34A.1Y, JP1.25; no longer IC89A.1Y, JP2.25
- net ADRR_13: now also IC34A.2Y, JP1.27; no longer IC89A.2Y, JP2.27
- net ADRR_14: now also IC34A.3Y, JP1.29; no longer IC89A.3Y, JP2.29
- net ADRR_15: now also IC34A.4Y, IC67C.I, IC68C.I0; no longer IC17C.I0, IC35C.I, IC89A.4Y
- net ADRR_2: now also IC13A.3Y, JP1.5; no longer IC86A.3Y, JP2.5
- net ADRR_3: now also IC13A.4Y, JP1.7; no longer IC86A.4Y, JP2.7
- net ADRR_4: now also IC21A.1Y, JP1.9; no longer IC87A.1Y, JP2.9
- net ADRR_5: now also IC21A.2Y, JP1.11; no longer IC87A.2Y, JP2.11
- net ADRR_6: now also IC21A.3Y, JP1.13; no longer IC87A.3Y, JP2.13
- net ADRR_7: now also IC21A.4Y, JP1.15; no longer IC87A.4Y, JP2.15
- net ADRR_8: now also IC27A.1Y, JP1.17; no longer IC88A.1Y, JP2.17
- net ADRR_9: now also IC27A.2Y, JP1.19; no longer IC88A.2Y, JP2.19
- net ALU_CARRY_BIT: now also IC55B.Q, IC62B.I0, JP4.16; no longer IC15B.Q, IC34B.I0, JP1.16
- net ALU_CARRY_IN: now also IC62B.O; no longer IC34B.O
- net ALU_CARRY_OUT: now also IC109D.I0, IC55B.D, IC88C.I0; no longer IC101C.I0, IC15B.D, IC31D.I0
- net ALU_NR1_ENABLE_ALU: now also IC49C.I0, IC70A.I0, IC77A.O; no longer IC18A.O, IC191A.I0, IC25C.I0
- net ALU_NR1_ENABLE_JMP_O_PTR_ADD: now also IC49C.I1, IC59C.O; no longer IC127C.O, IC25C.I1
- net ALU_NR2_ENABLE_ALU: now also IC49D.I0, IC70A.I1, IC77B.O; no longer IC18B.O, IC191A.I1, IC25D.I0
- net ALU_NR2_ENABLE_JMP_O_PTR_ADD: now also IC108C.O, IC49D.I1; no longer IC125C.O, IC25D.I1
- net ALU_NR3_ENABLE_ALU: now also IC70B.I0, IC77C.O; no longer IC18C.O, IC191B.I0
- net ALU_NR4_ENABLE_ALU: now also IC70B.I1, IC77D.O; no longer IC18D.O, IC191B.I1
- net CLR_NOT_CS/FILL_REGISTER_LDR: now also IC105A.I0, IC107C.O, IC68B.I0, IC96B.I1; no longer IC108B.I1, IC173A.I0, IC17B.I0, IC27C.O
- net CLR_NOT_CS_POP/FILL_REGISTER_POP: now also IC108A.O, IC19C.I1, IC39D.I0, IC96B.I0; no longer IC108B.I0, IC125A.O, IC48D.I0, IC85C.I1
- net CLR_NOT_CS_PUSH: now also IC105B.I0, IC107A.O, IC19C.I0; no longer IC173B.I0, IC27A.O, IC85C.I0
- net CLR_NOT_CS_STR: now also IC105C.I0, IC107D.O, IC68A.I1; no longer IC173C.I0, IC17A.I1, IC27D.O
- net CLR_NOT_OE/CLR_NOT_CS_CYCL_1/2: now also IC19D.I0, IC68A.I0, IC84B.O; no longer IC17A.I0, IC80B.O, IC85D.I0
- net CLR_NOT_OE/CLR_NOT_CS_CYCL_3/4: now also IC68B.I1, IC84D.O; no longer IC17B.I1, IC80D.O
- net CLR_NOT_OE_POP: now also IC39D.O, JP2.4; no longer IC48D.O, JP3.4
- net CNNCT_PTR_TO_ABUS/CNNCT_REG_TO_DBUS/CLR_NOT_WE/SEL_2_STR: now also IC105C.O, IC17C.I0, IC40A.I1, IC67B.I; no longer IC173C.O, IC2C.I0, IC35B.I, IC36A.I1
- net CONNECT_PTR_TO_ABUS/CLR_NOT_OE_LDR: now also IC105A.O, IC19D.I1, IC40A.I0; no longer IC173A.O, IC36A.I0, IC85D.I1
- net CONNECT_REG_TO_DBUS/CLR_NOT_WE/SELECTOR_TABLE_2_PUSH: now also IC105B.O, IC17C.I1, IC67A.I; no longer IC173B.O, IC2C.I1, IC35A.I
- net CONNECT_REG_TO_DBUS_PTR/FILL_PTR_L_SET_PTR: now also IC39A.I1, IC61B.I0, IC99D.O; no longer IC24D.O, IC48A.I1, IC52B.I0
- net CYCL_1: now also IC52A.Q, IC52B.D, IC84B.I1, JP4.22; no longer IC10A.Q, IC10B.D, IC80B.I1, JP1.22
- net DATA0: now also IC101A.1Q, IC18A.1D, IC26A.1D, IC33A.1D, IC35A.1Q, IC36A.1Q, IC41A.1D, IC45A.1D, IC57A.A, IC5A.1D, IC60A.A, IC66A.1D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; no longer IC100A.1D, IC116A.1Q, IC179A.A, IC181A.A, IC42A.1Q, IC63A.1D, IC64A.1D, IC70A.1D, IC71A.1D, IC72A.1Q, IC77A.1A, IC82A.A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
- net DATA1: now also IC101A.2Q, IC18A.2D, IC26A.2D, IC33A.2D, IC35A.2Q, IC36A.2Q, IC41A.2D, IC45A.2D, IC57A.B, IC5A.2D, IC60A.B, IC66A.2D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; no longer IC100A.2D, IC116A.2Q, IC179A.B, IC181A.B, IC42A.2Q, IC63A.2D, IC64A.2D, IC70A.2D, IC71A.2D, IC72A.2Q, IC77A.2A, IC82A.B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
- net DATA2: now also IC101A.3Q, IC18A.3D, IC26A.3D, IC33A.3D, IC35A.3Q, IC36A.3Q, IC41A.3D, IC45A.3D, IC57A.C, IC5A.3D, IC60A.C, IC66A.3D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; no longer IC100A.3D, IC116A.3Q, IC179A.C, IC181A.C, IC42A.3Q, IC63A.3D, IC64A.3D, IC70A.3D, IC71A.3D, IC72A.3Q, IC77A.3A, IC82A.C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
- net DATA3: now also IC101A.4Q, IC18A.4D, IC26A.4D, IC33A.4D, IC35A.4Q, IC36A.4Q, IC41A.4D, IC45A.4D, IC57A.D, IC5A.4D, IC60A.D, IC66A.4D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; no longer IC100A.4D, IC116A.4Q, IC179A.D, IC181A.D, IC42A.4Q, IC63A.4D, IC64A.4D, IC70A.4D, IC71A.4D, IC72A.4Q, IC77A.4A, IC82A.D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
- net DATA4: now also IC101A.5Q, IC104A.1A, IC18A.5D, IC26A.5D, IC33A.5D, IC35A.5Q, IC36A.5Q, IC41A.5D, IC45A.5D, IC58A.A, IC5A.5D, IC64A.A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; no longer IC100A.5D, IC116A.5Q, IC180A.A, IC182A.A, IC42A.5Q, IC63A.5D, IC64A.5D, IC70A.5D, IC71A.5D, IC72A.5Q, IC79A.1A, IC83A.A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
- net DATA5: now also IC101A.6Q, IC104A.2A, IC18A.6D, IC26A.6D, IC33A.6D, IC35A.6Q, IC36A.6Q, IC41A.6D, IC45A.6D, IC58A.B, IC5A.6D, IC64A.B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; no longer IC100A.6D, IC116A.6Q, IC180A.B, IC182A.B, IC42A.6Q, IC63A.6D, IC70A.6D, IC71A.6D, IC72A.6Q, IC79A.2A, IC83A.B, IC84A.6D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
- net DATA6: now also IC101A.7Q, IC104A.3A, IC18A.7D, IC26A.7D, IC33A.7D, IC35A.7Q, IC36A.7Q, IC41A.7D, IC45A.7D, IC58A.C, IC5A.7D, IC64A.C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; no longer IC100A.7D, IC116A.7Q, IC180A.C, IC182A.C, IC42A.7Q, IC63A.7D, IC64A.6D, IC64A.7D, IC70A.7D, IC71A.7D, IC72A.7Q, IC79A.3A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
- net DATA7: now also IC101A.8Q, IC104A.4A, IC18A.8D, IC26A.8D, IC33A.8D, IC35A.8Q, IC36A.8Q, IC41A.8D, IC45A.8D, IC58A.D, IC5A.8D, IC64A.D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; no longer IC100A.8D, IC116A.8Q, IC180A.D, IC182A.D, IC42A.8Q, IC63A.8D, IC64A.8D, IC70A.8D, IC71A.8D, IC72A.8Q, IC79A.4A, IC83A.D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
- net DATA_BUS_ENABLE_LATCH: now also IC35A.ENC, IC59A.O, IC67D.I; no longer IC127A.O, IC35D.I, IC72A.ENC
- net DBUS_SELECTOR_TABLE_2: now also IC11A.!A!/B, IC17C.O, IC63A.I0; no longer IC110A.I0, IC2C.O, IC46A.!A!/B
- net FDSGDFGFDSGFSDGFDGSDG: now also IC19A.O, IC8C.I1, IC8D.I1; no longer IC22C.I1, IC22D.I1, IC85A.O
- net FSDFAFSDFSFDDDDDDDDDDDDDDDDDDDDDDDDDDDDDDDD1: now also IC10A.I1, IC10C.I1, IC20B.O, IC2A.I1, IC2C.I1; no longer IC136B.O, IC39A.I1, IC39C.I1, IC41A.I1, IC41C.I1
- net GND: now also C108.2, C24.2, C25.2, C37.2, C41.2, C45.2, C46.2, C54.2, C62.2, C66.2, C69.2, C76.2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; no longer C117.2, C120.2, C121.2, C122.2, C123.2, C127.2, C142.2, C143.2, C145.2, C148.2, C150.2, C151.2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
- net HGGJHGGJZGZ77UZGHGHHGHGHGHGHJGHJ: now also IC100C.O, IC105A.I1; no longer IC173A.I1, IC51C.O
- net INPUT_REG0/OPC4/5_IS_NULL: now also IC109B.I1, IC24A.I0, IC24B.I0, IC28A.O, IC2A.I0, IC2B.I0, IC88A.I0, IC9A.1B; no longer IC101A.I0, IC126A.1B, IC129A.O, IC135A.I0, IC135B.I0, IC31B.I1, IC41A.I0, IC41B.I0
- net INPUT_REG1: now also IC24C.I0, IC24D.I0, IC28B.O, IC2C.I0, IC2D.I0, IC9A.2B; no longer IC126A.2B, IC129B.O, IC135C.I0, IC135D.I0, IC41C.I0, IC41D.I0
- net INPUT_REG2: now also IC10A.I0, IC10B.I0, IC28C.O, IC9A.3B; no longer IC126A.3B, IC129C.O, IC39A.I0, IC39B.I0
- net INPUT_REG3: now also IC10C.I0, IC10D.I0, IC28D.O, IC9A.4B; no longer IC126A.4B, IC129D.O, IC39C.I0, IC39D.I0
- net INPUT_REG_IS_NOT_OUTPUT_REG: now also IC17B.O, IC19A.I1, IC6A.I0, IC6B.I0, IC6C.I0, IC6D.I0, IC96C.I0; no longer IC108C.I0, IC2B.O, IC4A.I0, IC4B.I0, IC4C.I0, IC4D.I0, IC85A.I1
- net IO_INPUT1_0: now also IC3A.D7, JP3.2; no longer IC61A.D7, JP10.2
- net IO_INPUT1_1: now also IC15A.D7, JP3.4; no longer IC60A.D7, JP10.4
- net IO_INPUT1_2: now also IC22A.D7, JP3.6; no longer IC59A.D7, JP10.6
- net IO_INPUT1_3: now also IC31A.D7, JP3.8; no longer IC58A.D7, JP10.8
- net IO_INPUT1_4: now also IC37A.D7, JP3.10; no longer IC57A.D7, JP10.10
- net IO_INPUT1_5: now also IC42A.D7, JP3.12; no longer IC56A.D7, JP10.12
- net IO_INPUT1_6: now also IC46A.D7, JP3.14; no longer IC3A.D7, JP10.14
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Other:
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
Commit message: fix WRITE_TO_DBUS signal
Parts:
- removed IC107, IC62: 74HCT08N, 74xx-eu:74HCT08N
- removed IC63: 74HCT32N, 74xx-eu:74HCT32N
- added IC112: 74HCT32N, 74xx-eu:74HCT32N
- added IC118, IC131: 74HC74N, 74xx-eu:74HC74N
- added IC125, IC126, IC130: 74HCT08N, 74xx-eu:74HCT08N
- added IC129: 74HCT04N, 74xx-eu:74HCT04N
- IC105: value 74HCT32N -> 74HC74N; device 74xx-eu:74HCT32N -> 74xx-eu:74HC74N
- IC52: value 74HC74N -> 74HCT08N; device 74xx-eu:74HC74N -> 74xx-eu:74HCT08N
- IC55: value 74HC74N -> 74HCT32N; device 74xx-eu:74HC74N -> 74xx-eu:74HCT32N
Connections:
- net N$32 renamed REG_TO_DBUS_L_JMP_RET
- net N$33 renamed REG_TO_DBUS_H_JMP_RET
- removed net CLR_NOT_CS/FILL_REGISTER_LDR: IC105A.I0, IC107C.O, IC68B.I0, IC96B.I1
- removed net CLR_NOT_CS_POP/FILL_REGISTER_POP: IC108A.O, IC19C.I1, IC39D.I0, IC96B.I0
- removed net CLR_NOT_CS_PUSH: IC105B.I0, IC107A.O, IC19C.I0
- removed net CLR_NOT_CS_STR: IC105C.I0, IC107D.O, IC68A.I1
- removed net CLR_NOT_OE/CLR_NOT_CS_CYCL_1/2: IC19D.I0, IC68A.I0, IC84B.O
- removed net CLR_NOT_OE/CLR_NOT_CS_CYCL_3/4: IC68B.I1, IC84D.O
- removed net CLR_NOT_OE_POP: IC39D.O, JP2.4
- removed net CNNCT_PTR_TO_ABUS/CNNCT_REG_TO_DBUS/CLR_NOT_WE/SEL_2_STR: IC105C.O, IC17C.I0, IC40A.I1, IC67B.I
- removed net CONNECT_PTR_TO_ABUS/CLR_NOT_OE_LDR: IC105A.O, IC19D.I1, IC40A.I0
- removed net CONNECT_REG_TO_DBUS/CLR_NOT_WE/SELECTOR_TABLE_2_PUSH: IC105B.O, IC17C.I1, IC67A.I
- removed net CONNECT_REG_TO_DBUS_PTR/FILL_PTR_L_SET_PTR: IC39A.I1, IC61B.I0, IC99D.O
- removed net CYCL_1: IC52A.Q, IC52B.D, IC84B.I1, JP4.22
- removed net HGGJHGGJZGZ77UZGHGHHGHGHGHGHJGHJ: IC100C.O, IC105A.I1
- removed net IR_LOAD_INPUT/PC_COUNT_UP_FETCH2/CYCL_4: IC41A.CLK, IC49A.I0, IC53B.Q, IC56A.I1, IC84D.I0, JP4.28
- removed net LATCH_ALU_INPUT_B_ALU: IC63D.I0, IC71A.I0, IC72A.O
- removed net LATCH_ALU_INPUT_B_JMP_O: IC63C.I0, IC78D.O, IC84A.I0
- removed net LATCH_ALU_INPUT_B_PTR_ADD: IC105D.I0, IC63C.I1, IC89A.O
- removed net N$109: IC76D.O, IC84A.I1
- removed net N$110: IC71A.I1, IC76B.O
- removed net N$123: IC100D.O, IC105C.I1
- removed net N$132: IC108B.O, IC71B.I0, IC72D.I1, IC76D.I1, IC78D.I1
- removed net N$146: IC105B.I1, IC107B.O
- removed net N$151: IC105D.I1, IC99B.O
- removed net N$152: IC63C.O, IC63D.I1
- removed net N$157: IC100B.O, IC39D.I1
- removed net OPCODE_LOAD_INPUT/CYCL_2: IC45A.CLK, IC52B.Q, IC53A.D, IC84B.I0, JP4.24
- removed net PC_COUNT_UP_FETCH1/CYCL_3: IC53B.D, IC56A.I0, IC84D.I1, IC89D.O, JP4.26
- removed net PTR_ADD_OR_JMP_O_OR_ALU_FILL: IC14D.I, IC1B.I0, IC1C.O
- removed net STATE_0/CYCL_5: IC100B.I0, IC100C.I0, IC100D.I0, IC109C.I0, IC54A.Q, IC54B.D, IC76A.I0, IC76B.I0, IC76C.I0, IC76D.I0, IC99A.I0, IC99B.I0, IC99C.I0, IC99D.I0, JP4.30
- removed net STATE_1/CYCL_6: IC100A.I0, IC107B.I0, IC107C.I0, IC107D.I0, IC108A.I0, IC54B.Q, IC55A.D, IC72A.I0, IC72C.I0, IC78D.I0, IC89A.I0, IC92A.I0, IC92B.I0, JP4.32
- removed net STATE_2/CYCL_7: IC107A.I0, IC109A.I0, IC52A.D, IC55A.Q, IC72B.I0, IC72D.I0, IC89B.I0, JP4.34
- removed net WRITE_LR_H_DBUS/FILL_PC_H_RET: IC100A.O, IC40B.I0, IC56B.I0, IC65A.I1
- removed net WRITE_LR_L_DBUS_RET/FILL_PC_L_RET: IC56C.I1, IC65A.I0, IC99A.O
- removed net WRITE_PC_H_DBUS/FILL_LR_H_SAVE_LR: IC44D.I0, IC65D.I1, IC92B.O
- removed net WRITE_PC_L_DBUS/FILL_LR_L_SAVE_LR: IC40B.I1, IC44C.I0, IC65D.I0, IC99C.O
- removed net WRITE_REGB_TO_DBUS/FILL_PC_L_JMP_O: IC1A.I1, IC56D.I0, IC72D.O, IC88C.I1
- removed net WRITE_REGB_TO_DBUS/FILL_PTR_H_SET_PTR: IC1D.I1, IC39B.I1, IC92A.O
- removed net WRITE_REGB_TO_DBUS/FILL_PTR_L_PTR_ADD: IC109D.I1, IC1A.I0, IC72B.O
- removed net WRITE_REGB_TO_DBUS/FILL_REGISTER/ALU_TO_DBUS_ALU: IC17D.I1, IC1C.I1, IC55B.CLK, IC89B.O
- removed net WRITE_REGB_TO_DBUS/PC_HIGH_LOAD_INPUT_JMP: IC1D.I0, IC44B.I0, IC72C.O
- removed net WRITE_REG_TO_DBUS_JMP/PC_LOW_LOAD_INPUT_JMP: IC56C.I0, IC61A.I0, IC76C.O
- removed net WRITE_REG_TO_DBUS_MOV/FILL_REGISTER_MOV: IC17D.I0, IC61B.I1, IC76A.O
- new net !ENABLE_REG_OUTPUT: IC112A.I0, IC55D.O, IC84B.I1
- new net ALU_OUTPUT_ENABLE/FILL_PC_L_JMP_O: IC112B.I1, IC56D.I0, IC72D.O, IC88C.I1
- new net ALU_OUTPUT_ENABLE/FILL_PTR_L_PTR_ADD: IC109D.I1, IC1A.I0, IC55A.I1, IC72B.O
- new net CARRY_LAST_CYCLE: IC109D.I0, IC118B.Q, IC88C.I0
- new net CLR_NOT_OE/CLR_NOT_CS_CYCL_1: IC19D.I0, IC53A.Q, IC55B.I1, IC68A.I0, IC89C.I0, IC89D.I0, JP4.26
- new net CLR_NOT_OE/CLR_NOT_CS_CYCL_2: IC49A.I0, IC53B.Q, IC55B.I0, IC68B.I1, JP4.28
- new net CLR_NOT_OE/CLR_NOT_CS_POP/FILL_REGISTER_POP: IC100B.O, IC19C.I1, IC96B.I0, JP2.4
- new net ENABLE_ALU_OUTPUT: IC14D.I, IC55A.O, IC55C.I1
- new net ENABLE_ALU_OUTPUT/FILL_REGISTER_ALU: IC112B.I0, IC17D.I1, IC52B.O
- new net IR_LOAD_INPUT/PC_COUNT_UP/!CYCL_2: IC41A.CLK, IC49B.I1, IC53B.!Q
- new net LATCH_ALU_INPUT_B/WRITE_REGB_TO_DBUS_JMP_O: IC1A.I1, IC76D.O, IC84D.I0
- new net N$18: IC53B.D, IC89D.O
- new net N$32: IC55C.O, IC55D.I1
- new net N$33: IC55B.O, IC55D.I0
- new net N$74: IC118A.CLK, IC129A.O
- new net N$79: IC112C.O, IC112D.I0
- new net N$81: IC129D.O, IC129E.I
- new net N$83: IC129E.O, IC129F.I
- new net N$84: IC129F.O, IC130A.I1
- new net N$85: IC131B.Q, IC84B.I0
- new net N$86: IC112B.O, IC55A.I0
- new net N$87: IC130A.O, IC131B.CLK
- new net N$88: IC112A.I1, IC131B.!Q
- new net N$89: IC101A.OC, IC14D.O
- new net N$91: IC1B.I0, IC1C.O
- new net OPCODE_LOAD_INPUT/PC_COUNT_UP/!CYCL_1: IC45A.CLK, IC49B.I0, IC53A.!Q
- new net REG_TO_DBUS_B_ALU_PTR_ADD: IC84A.O, IC84D.I1
- new net REG_TO_DBUS_ENABLE/CLR_NOT_CS/CLR_NOT_WE_PUSH: IC126B.O, IC19C.I0, IC67A.I
- new net REG_TO_DBUS_ENABLE/FILL_LR_H_SAVE_LR: IC125B.O, IC44D.I0
- new net REG_TO_DBUS_ENABLE/FILL_LR_L_SAVE_LR: IC44C.I0, IC92B.O
- new net REG_TO_DBUS_ENABLE/FILL_PC_H_RET: IC126C.O, IC56B.I0
- new net REG_TO_DBUS_ENABLE/FILL_PC_L_RET: IC100A.O, IC56C.I1
- new net REG_TO_DBUS_ENABLE/FILL_PTR_H_SET_PTR: IC125D.O, IC39B.I1
- new net REG_TO_DBUS_ENABLE/FILL_PTR_L_SET_PTR: IC39A.I1, IC92A.O
- new net REG_TO_DBUS_ENABLE/FILL_REGISTER_MOV: IC108A.O, IC17D.I0
- new net REG_TO_DBUS_ENABLE/LATCH_ALU_INPUT_B/WRITE_REGB_TO_DBUS_ALU: IC1C.I1, IC72A.O, IC84A.I0
- new net REG_TO_DBUS_ENABLE/LATCH_ALU_INPUT_B/WRITE_REGB_TO_DBUS_PTR_ADD: IC84A.I1, IC89A.O
- new net REG_TO_DBUS_ENABLE/PC_HIGH_LOAD_INPUT_JMP: IC52C.O, IC56B.I1
- new net REG_TO_DBUS_ENABLE/PC_LOW_LOAD_INPUT_JMP: IC56C.I0, IC72C.O
- new net REG_TO_DBUS_ENABLE/STORE_ALU_OUTPUT/STORE_CARRY_ALU: IC112C.I0, IC129A.I, IC52A.O
- new net REG_TO_DBUS_ENABLE/STORE_ALU_OUTPUT/STORE_CARRY_TMP_JMP_O: IC112C.I1, IC39D.I0, IC78D.O
- new net REG_TO_DBUS_ENABLE/STORE_ALU_OUTPUT/STORE_CARRY_TMP_PTR_ADD: IC112D.I1, IC125A.O, IC39D.I1
- new net REG_TO_DBUS_ENABLE/WRITE_PTR_TO_ABUS/CLR_NOT_WE/CLR_NOT_CS_STR: IC130C.O, IC40A.I1, IC67B.I, IC68A.I1
- new net STATE_0/CYCL_3: IC100B.I0, IC100C.I0, IC100D.I0, IC130B.I0, IC54A.Q, IC54B.D, IC76A.I0, IC76B.I0, IC76C.I0, IC76D.I0, IC99A.I0, IC99B.I0, IC99C.I0, IC99D.I0, JP4.30
- new net STATE_1/CYCL_4: IC100A.I0, IC105A.D, IC108A.I0, IC109A.I0, IC126B.I0, IC130C.I0, IC54B.Q, IC72A.I0, IC72C.I0, IC78D.I0, IC89A.I0, IC92A.I0, IC92B.I0, JP4.32
- new net STATE_2/CYCL_5: IC105A.Q, IC105B.D, IC125A.I0, IC125C.I0, IC126A.I0, IC126D.I0, IC52A.I0, IC52D.I0, IC72D.I0, JP4.34
- new net STATE_3/CYCL_6: IC105B.Q, IC125B.I0, IC125D.I0, IC126C.I0, IC52B.I0, IC52C.I0, IC53A.D, IC72B.I0
- new net STORE_ALU_OUTPUT: IC101A.ENC, IC112D.O
- new net WRITE_LR_H_DBUS_RET: IC126A.O, IC40B.I0, IC65A.I1
- new net WRITE_LR_L_DBUS_RET: IC65A.I0, IC99A.O
- new net WRITE_PC_H_DBUS_SAVE_LR: IC126D.O, IC65D.I1
- new net WRITE_PC_L_DBUS_SAVE_LR: IC40B.I1, IC65D.I0, IC99C.O
- new net WRITE_PTR_TO_ABUS/CLR_NOT_OE/CLR_NOT_CS/FILL_REGISTER_LDR: IC100C.O, IC19D.I1, IC40A.I0, IC55C.I0, IC68B.I0, IC96B.I1
- new net WRITE_REGB_TO_DBUS_JMP: IC1D.I0, IC52D.O
- new net WRITE_REGB_TO_DBUS_SET_PTR: IC125C.O, IC1D.I1
- new net WRITE_REG_TO_DBUS_JMP: IC61A.I0, IC76C.O
- new net WRITE_REG_TO_DBUS_MOV: IC61B.I1, IC76A.O
- new net WRITE_REG_TO_DBUS_SELECTOR2_PUSH: IC130B.O, IC17C.I1, IC67D.I
- new net WRITE_REG_TO_DBUS_SELECTOR2_STR: IC100D.O, IC17C.I0
- new net WRITE_REG_TO_DBUS_SET_PTR: IC61B.I0, IC99D.O
- net !CLR_CARRY_BIT: now also IC118A.CLR; no longer IC55B.CLR
- net !RING_CNTR_RESET: now also IC105A.CLR, IC105B.CLR, IC53A.PRE; no longer IC52A.PRE, IC52B.CLR, IC53A.CLR, IC55A.CLR
- net !SET_CARRY_BIT: now also IC118A.PRE; no longer IC55B.PRE
- net ALU_CARRY_BIT: now also IC118A.Q, IC89B.I0; no longer IC55B.Q, IC62B.I0
- net ALU_CARRY_IN: now also IC89B.O; no longer IC62B.O
- net ALU_CARRY_OUT: now also IC118A.D, IC118B.D; no longer IC109D.I0, IC55B.D, IC88C.I0
- net DATA_BUS_ENABLE_LATCH: no longer IC67D.I
- net DBUS_SELECTOR_TABLE_2: now also IC56A.I0; no longer IC63A.I0
- net GND: now also JP4.22, JP4.24
- net LDR: no longer IC107C.I1
- net N$12: no longer IC67E.I
- net N$14: now also IC118B.CLK, IC39D.O; no longer IC101A.ENC, IC101A.OC, IC14D.O
- net N$15: now also IC52C.I1, IC52D.I1
- net N$190: now also IC94A.I1; no longer IC96A.I1
- net N$192: now also IC94A.I0, IC96A.O; no longer IC94A.O, IC96A.I0
- net N$193: now also IC94A.O; no longer IC96A.O
- net N$194: now also IC125B.I1, IC126D.I1
- net N$2: now also IC56A.O, IC71A.I0; no longer IC63A.O, IC63B.I0
- net N$219: now also IC126A.I1, IC126C.I1
- net N$266: now also IC129C.I
- net N$44: now also IC112A.O, IC36A.OC; no longer IC53A.Q, IC89C.I0, IC89D.I0
- net N$52: now also IC129C.O, IC129D.I, IC130A.I0; no longer IC36A.OC, IC67E.O
- net N$55: now also IC108A.I1
- net N$7: now also IC129B.O; no longer IC67F.O
- net N$90: now also IC71A.O; no longer IC63B.O
- net N$96: now also IC84D.O; no longer IC63D.O
- net N$97: now also IC125C.I1, IC125D.I1
- net OPERAND_REGB_OUTPUT: now also IC56A.I1; no longer IC63A.I1
- net PC_COUNT_UP: now also IC49B.O; no longer IC56A.O
- net PC_H_LOAD_INPUT_TABLE_1: now also IC44B.I0; no longer IC56B.I1
- net POP: no longer IC108A.I1
- net PTR_ADD: now also IC125A.I1
- net PUSH: now also IC126B.I1, IC130B.I1; no longer IC107A.I1, IC107B.I1, IC109C.I1
- net REGISTER_OUTPUT_SEL_3: now also IC129B.I, IC131B.D; no longer IC67F.I
- net REGS_OUTPUT_TO_DATABUS_ENABLE: now also IC84B.O; no longer IC67D.O
- net REG_0_OUT_0: now also IC96A.I0; no longer IC94A.I0
- net REG_0_OUT_1: now also IC96A.I1; no longer IC94A.I1
- net RING_CNTR_CLOCK: now also IC105A.CLK, IC105B.CLK; no longer IC52A.CLK, IC52B.CLK, IC55A.CLK
- net SELECT_CARRY_BIT: now also IC52A.I1, IC52B.I1; no longer IC62B.I1
- net SP_COUNT_UP: now also IC67D.O; no longer IC109C.O
- net STR: now also IC130C.I1; no longer IC107D.I1
- net VCC: now also IC105A.PRE, IC105B.PRE, IC118B.CLR, IC118B.PRE, IC131B.CLR, IC131B.PRE, IC53A.CLR; no longer IC52A.CLR, IC52B.PRE, IC53A.PRE, IC55A.PRE
- net WRITE_PC_L_ALU_LATCH_JMP_O: now also IC108B.O, IC71B.I0, IC72D.I1, IC76D.I1, IC78D.I1; no longer IC84A.O
- net WRITE_PTR_L_TO_DBUS_PTR_ADD: now also IC71A.I1, IC99B.O; no longer IC105D.O, IC63B.I1
- net WRITE_REG_TO_DBUS_ALU: now also IC76B.O; no longer IC71A.O
Other:
- note added: "CYCL_1"
- note added: "When ALU, LDR, OR FETCH is active --> DONT output reg to DBUS"
- note removed: "CYCL_3"
- note removed: "CYCL_7"
- note removed: "Do we need a pause between both CS/Read Cycles?"
- note removed: "Does this work? Is there enough time?"
- note removed: "I am not happy with the memory. Too much FLash and too little RAM"
- note removed: "Maybe we can omit the first FF and do the SIgnal int Cycl7"
- moved on the sheet: IC100A, IC100B, IC100C, IC100D, IC101, IC108A, IC108B, IC108C, IC108D, IC109A, IC109C, IC109D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

Commit message: optimize part count
Parts:
- removed IC104, IC98: 74ACT157N, 74xx-eu:74ACT157N
- removed IC109: 74HCT00N, 74xx-eu:74HCT00N
- removed IC125, IC76: 74HCT08N, 74xx-eu:74HCT08N
- removed IC61, IC84: 74HCT32N, 74xx-eu:74HCT32N
- added IC62: 74HCT08N, 74xx-eu:74HCT08N
- IC40: value 74HCT32N -> 74HCT08N; device 74xx-eu:74HCT32N -> 74xx-eu:74HCT08N
Connections:
- net REG_TO_DBUS_ENABLE/CLR_NOT_CS/CLR_NOT_WE_PUSH renamed CLR_NOT_CS/CLR_NOT_WE_PUSH
- net REG_TO_DBUS_ENABLE/FILL_REGISTER_MOV renamed FILL_REGISTER_MOV
- net REG_TO_DBUS_ENABLE/PC_HIGH_LOAD_INPUT_JMP renamed PC_HIGH_LOAD_INPUT_JMP
- removed net CLR_NOT_OE/CLR_NOT_CS_CYCL_1: IC19D.I0, IC53A.Q, IC55B.I1, IC68A.I0, IC89C.I0, IC89D.I0, JP4.26
- removed net CLR_NOT_OE/CLR_NOT_CS_CYCL_2: IC49A.I0, IC53B.Q, IC55B.I0, IC68B.I1, JP4.28
- removed net IR_LOAD_INPUT/PC_COUNT_UP/!CYCL_2: IC41A.CLK, IC49B.I1, IC53B.!Q
- removed net N$108: IC103A.2D, IC98A.2Y
- removed net N$114: IC103A.3D, IC98A.3Y
- removed net N$116: IC103A.4D, IC98A.4Y
- removed net N$121: IC61C.O, IC61D.I0
- removed net N$124: IC103A.5D, IC104A.1Y
- removed net N$125: IC103A.6D, IC104A.2Y
- removed net N$126: IC19B.I0, IC68A.O
- removed net N$127: IC103A.7D, IC104A.3Y
- removed net N$134: IC103A.8D, IC104A.4Y
- removed net N$139: IC88B.I1, IC88C.O, IC88D.I1
- removed net N$150: IC61B.O, IC61C.I1
- removed net N$154: IC61A.O, IC61C.I0
- removed net N$159: IC109D.O, IC40C.I1, IC40D.I1
- removed net N$17: IC103A.1D, IC98A.1Y
- removed net N$200: IC19B.I1, IC68B.O
- removed net N$252: IC61D.I1, IC65B.O
- removed net N$266: IC129C.I, IC59A.I1, IC59D.I1, IC61D.O
- removed net N$32: IC55C.O, IC55D.I1
- removed net N$33: IC55B.O, IC55D.I0
- removed net N$79: IC112C.O, IC112D.I0
- removed net N$90: IC65B.I0, IC71A.O
- removed net N$91: IC1B.I0, IC1C.O
- removed net N$96: IC103A.ENC, IC84D.O
- removed net OPCODE_LOAD_INPUT/PC_COUNT_UP/!CYCL_1: IC45A.CLK, IC49B.I0, IC53A.!Q
- removed net PTR_TO_ABUS/!PC_TO_ABUS: IC13A.!A!/B, IC21A.!A!/B, IC27A.!A!/B, IC34A.!A!/B, IC40A.O
- removed net REG_TO_DBUS_B_ALU_PTR_ADD: IC84A.O, IC84D.I1
- removed net REG_TO_DBUS_ENABLE/FILL_LR_H_SAVE_LR: IC125B.O, IC44D.I0
- removed net REG_TO_DBUS_ENABLE/FILL_LR_L_SAVE_LR: IC44C.I0, IC92B.O
- removed net REG_TO_DBUS_ENABLE/FILL_PC_H_RET: IC126C.O, IC56B.I0
- removed net REG_TO_DBUS_ENABLE/FILL_PC_L_RET: IC100A.O, IC56C.I1
- removed net REG_TO_DBUS_ENABLE/FILL_PTR_H_SET_PTR: IC125D.O, IC39B.I1
- removed net REG_TO_DBUS_ENABLE/FILL_PTR_L_SET_PTR: IC39A.I1, IC92A.O
- removed net REG_TO_DBUS_ENABLE/LATCH_ALU_INPUT_B/WRITE_REGB_TO_DBUS_ALU: IC1C.I1, IC72A.O, IC84A.I0
- removed net REG_TO_DBUS_ENABLE/LATCH_ALU_INPUT_B/WRITE_REGB_TO_DBUS_PTR_ADD: IC84A.I1, IC89A.O
- removed net REG_TO_DBUS_ENABLE/PC_LOW_LOAD_INPUT_JMP: IC56C.I0, IC72C.O
- removed net REG_TO_DBUS_ENABLE/STORE_ALU_OUTPUT/STORE_CARRY_ALU: IC112C.I0, IC129A.I, IC52A.O
- removed net REG_TO_DBUS_ENABLE/STORE_ALU_OUTPUT/STORE_CARRY_TMP_JMP_O: IC112C.I1, IC39D.I0, IC78D.O
- removed net REG_TO_DBUS_ENABLE/STORE_ALU_OUTPUT/STORE_CARRY_TMP_PTR_ADD: IC112D.I1, IC125A.O, IC39D.I1
- removed net REG_TO_DBUS_ENABLE/WRITE_PTR_TO_ABUS/CLR_NOT_WE/CLR_NOT_CS_STR: IC130C.O, IC40A.I1, IC67B.I, IC68A.I1
- removed net SP_COUNT_UP: IC67D.O, IC93A.UP
- removed net WRITE_LR_H_DBUS_RET: IC126A.O, IC40B.I0, IC65A.I1
- removed net WRITE_PC_H_DBUS_SAVE_LR: IC126D.O, IC65D.I1
- removed net WRITE_PC_L_ALU_LATCH_JMP_O: IC104A.!A!/B, IC108B.O, IC71B.I0, IC72D.I1, IC76D.I1, IC78D.I1, IC98A.!A!/B
- removed net WRITE_REGB_TO_DBUS_SET_PTR: IC125C.O, IC1D.I1
- removed net WRITE_REG_TO_DBUS_ALU: IC61A.I1, IC76B.O
- removed net WRITE_REG_TO_DBUS_JMP: IC61A.I0, IC76C.O
- removed net WRITE_REG_TO_DBUS_MOV: IC61B.I1, IC76A.O
- removed net WRITE_REG_TO_DBUS_SELECTOR2_PUSH: IC130B.O, IC17C.I1, IC67D.I
- removed net WRITE_REG_TO_DBUS_SET_PTR: IC61B.I0, IC99D.O
- new net CARRY&&!IR_DATA: IC62A.O, IC62B.I0, IC88D.I0
- new net CARRY&&IR_DATA: IC62C.O, IC62D.I0, IC88B.I0
- new net CLR_NOT_OE/CLR_NOT_CS/PC_COUNT_UP_CYCL_2: IC49A.I0, IC53B.Q, IC55B.I0, JP4.28
- new net CLR_NOT_OE/PC_COUNT_UP/CLR_NOT_CS_CYCL_1: IC53A.Q, IC55B.I1, IC89C.I0, IC89D.I0, JP4.26
- new net CYCLE1/CYLCE2: IC19B.I1, IC39D.I0, IC55B.O, IC71A.I0
- new net FILL_LR_H_SAVE_LR: IC126D.O, IC44D.I0
- new net FILL_LR_L/WRITE_PC_H_DBUS_SAVE_LR: IC44C.I0, IC65D.I1, IC92B.O
- new net FILL_PC_H_RET: IC126A.O, IC56B.I0
- new net FILL_PC_L/WRITE_LR_H_DBUS_RET: IC100A.O, IC49B.I0, IC56C.I1, IC65A.I1
- new net FILL_PTR_H_SET_PTR: IC39B.I1, IC88C.O
- new net FILL_PTR_L/WRITE_REGB_TO_DBUS_SET_PTR: IC1D.I1, IC39A.I1, IC92A.O
- new net IR_LOAD_INPUT/!CYCL_2: IC41A.CLK, IC53B.!Q
- new net LATCH_ALU_INPUT_ALU/JMP_O/PTR_ADD: IC103A.ENC, IC1B.I0, IC1C.O
- new net LATCH_ALU_INPUT_B/WRITE_REGB_TO_DBUS_ALU: IC1A.I0, IC72A.O
- new net LATCH_ALU_INPUT_B/WRITE_REGB_TO_DBUS_PTR_ADD: IC1C.I1, IC89A.O
- new net MEM_OE: IC55D.I0, IC67F.I, IC71A.O
- new net OPCODE_LOAD_INPUT/!CYCL_1: IC45A.CLK, IC53A.!Q
- new net PC_COUNT_UP_RET: IC126C.O, IC39D.I1
- new net PC_LOW_LOAD_INPUT_JMP: IC52B.O, IC56C.I0
- new net PC_L_TO_DBUS: IC49B.I1, IC56A.O, IC65D.I0
- new net PTR_TO_ABUS: IC13A.!A!/B, IC19B.I0, IC21A.!A!/B, IC27A.!A!/B, IC34A.!A!/B, IC68A.O
- new net SP_COUNT_UP/WRITE_REG_TO_DBUS_SELECTOR2_PUSH: IC130B.O, IC17C.I1, IC93A.UP
- new net STORE_ALU_OUTPUT/STORE_CARRY_ALU: IC112D.I0, IC129A.I, IC72C.O
- new net STORE_ALU_OUTPUT/STORE_CARRY_TMP_JMP_O: IC112C.I0, IC40D.O
- new net STORE_ALU_OUTPUT/STORE_CARRY_TMP_PTR_ADD: IC112C.I1, IC52A.O
- new net STORE_ALU_OUTPUT_JMP_PTR_ADD: IC112C.O, IC112D.I1, IC67E.I
- new net WQWJKDHSAAASDFXGHCJFDSAAS: IC108B.O, IC40A.I1, IC40B.I1, IC40C.I1, IC40D.I1, IC71B.I0
- new net WRITE_PC_L_DBUS_JMP_O: IC40C.O, IC56A.I1
- new net WRITE_PTR_TO_ABUS/CLR_NOT_WE/CLR_NOT_CS_STR: IC130C.O, IC67B.I, IC68A.I1
- net !ENABLE_REG_OUTPUT: now also IC65B.I1; no longer IC84B.I1
- net !IR_DATA_OUT_7: now also IC62A.I1; no longer IC40D.I0, IC88D.I0
- net ALU_CARRY_BIT: now also IC78D.I0; no longer IC78C.I0
- net ALU_OUTPUT_ENABLE/FILL_PC_L_JMP_O: now also IC40A.O, IC88B.I1, IC88D.I1; no longer IC72D.O, IC88C.I1
- net ALU_OUTPUT_ENABLE/FILL_PTR_L_PTR_ADD: now also IC62B.I1, IC62D.I1; no longer IC109D.I1, IC1A.I0
- net CARRY_LAST_CYCLE: now also IC62A.I0, IC62C.I1; no longer IC109D.I0, IC88C.I0
- net DATA0: now also IC103A.1D; no longer IC98A.1A
- net DATA1: now also IC103A.2D; no longer IC98A.2A
- net DATA2: now also IC103A.3D; no longer IC98A.3A
- net DATA3: now also IC103A.4D; no longer IC98A.4A
- net DATA4: now also IC103A.5D; no longer IC104A.1A
- net DATA5: now also IC103A.6D; no longer IC104A.2A
- net DATA6: now also IC103A.7D; no longer IC104A.3A
- net DATA7: now also IC103A.8D; no longer IC104A.4A
- net DBUS_SELECTOR_TABLE_2: no longer IC56A.I0
- net ENABLE_ALU_OUTPUT: now also IC55D.I1; no longer IC55C.I1
- net ENABLE_ALU_OUTPUT/FILL_REGISTER_ALU: now also IC72D.O; no longer IC52B.O
- net GND: no longer IC104A.G, IC98A.G
- net INPUT_REG0/OPC4/5_IS_NULL: now also IC99D.I1; no longer IC109B.I1
- net IR_DATA_OUT_7: now also IC62C.I0; no longer IC40C.I0, IC88B.I0
- net LATCH_ALU_INPUT_B/WRITE_REGB_TO_DBUS_JMP_O: now also IC40B.O; no longer IC76D.O, IC84D.I0
- net MEM_NOT_OE: now also IC67F.O; no longer IC19D.O
- net N$13: now also IC68B.O; no longer IC84C.O
- net N$14: now also IC67E.O; no longer IC39D.O
- net N$15: now also IC52B.I1; no longer IC72C.I1, IC76C.I1
- net N$171: now also IC49B.O; no longer IC40B.O
- net N$194: now also IC78C.I1; no longer IC125B.I1, IC99C.I1
- net N$198: now also IC78D.O; no longer IC78C.O
- net N$199: now also IC78D.I1; no longer IC78C.I1
- net N$2: now also IC67D.I, IC99D.O; no longer IC56A.O, IC71A.I0
- net N$203: now also IC67D.O; no longer IC109B.O
- net N$21: now also IC68B.I1, IC99D.I0; no longer IC109B.I0, IC84C.I1
- net N$55: no longer IC76A.I1
- net N$80: now also IC68B.I0; no longer IC84C.I0
- net N$85: now also IC65B.I0; no longer IC84B.I0
- net N$97: now also IC88C.I1; no longer IC125C.I1, IC125D.I1, IC99D.I1
- net OPERAND_REGB_OUTPUT: no longer IC56A.I1
- net PC_COUNT_UP: now also IC39D.O; no longer IC49B.O
- net PC_DATA_OUT_0: no longer IC98A.1B
- net PC_DATA_OUT_1: no longer IC98A.2B
- net PC_DATA_OUT_2: no longer IC98A.3B
- net PC_DATA_OUT_3: no longer IC98A.4B
- net PC_DATA_OUT_4: no longer IC104A.1B
- net PC_DATA_OUT_5: no longer IC104A.2B
- net PC_DATA_OUT_6: no longer IC104A.3B
- net PC_DATA_OUT_7: no longer IC104A.4B
- net POP: now also IC130D.I1; no longer IC109A.I1
- net PTR_ADD: now also IC52A.I1; no longer IC125A.I1
- net PTR_HIGH_COUNT_DOWN: now also IC62D.O; no longer IC40C.O
- net PTR_HIGH_COUNT_UP: now also IC62B.O; no longer IC40D.O
- net REGS_OUTPUT_TO_DATABUS_ENABLE: now also IC65B.O; no longer IC84B.O
- net RING_CNTR_CLOCK: now also IC129C.I, IC59A.I1, IC59D.I1
- net SECOND_LATCH_SELECT: no longer IC65B.I1
- net SELECT_CARRY_BIT: now also IC72C.I1, IC72D.I1; no longer IC52A.I1, IC52B.I1, IC76B.I1
- net SP_COUNT_DOWN: now also IC130D.O; no longer IC109A.O
- net STATE_0/CYCL_3: now also IC40C.I0, IC78C.I0; no longer IC76A.I0, IC76B.I0, IC76C.I0, IC76D.I0, IC99C.I0, IC99D.I0
- net STATE_1/CYCL_4: now also IC130D.I0, IC40B.I0, IC52B.I0; no longer IC109A.I0, IC72C.I0, IC78D.I0
- net STATE_2/CYCL_5: now also IC40D.I0, IC72C.I0, IC88C.I0; no longer IC125A.I0, IC125C.I0, IC72D.I0
- net STATE_3/CYCL_6: now also IC40A.I0, IC72D.I0; no longer IC125B.I0, IC125D.I0, IC52B.I0
- net WRITE_PC_L_DBUS_SAVE_LR: now also IC56A.I0, IC78C.O; no longer IC40B.I1, IC65D.I0, IC99C.O
- net WRITE_PTR_L_TO_DBUS_PTR_ADD: no longer IC71A.I1
- net WRITE_PTR_TO_ABUS/CLR_NOT_OE/CLR_NOT_CS/FILL_REGISTER_LDR: now also IC68A.I0, IC71A.I1; no longer IC19D.I1, IC40A.I0, IC55C.I0, IC68B.I0
Other:
- note added: "Needs to count up twice actually"
- note added: "When ALU or Memory write to DBUS --> Dont output reg to dbus"
- note added: "Write reg to dbus in every cycle"
- note added: "only change latch on falling edge"
- note removed: "When ALU, LDR, OR FETCH is active --> DONT output reg to DBUS"
- moved on the sheet: IC101, IC103, IC112B, IC112C, IC112D, IC118A, IC118B, IC126A, IC126C, IC126D, IC129A, IC129B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
