File: schematics/Control_Unit/Control_Unit.sch (EAGLE design)
At the start: 220 parts, among them IC1 74HCT32N, IC10 74HCT08N, IC100 74HCT08N, IC101 74HC373N, IC102 74HC193N, IC103 74HC373N, IC105 74HC74N, IC106 74HC193N, IC108 74HCT08N, IC11 74ACT157N, IC112 74HCT32N, IC118 74HC74N, IC12 74ACT157N, IC126 74HCT08N, IC129 74HCT04N, IC13 74ACT157N, IC130 74HCT08N, IC131 74HC74N, IC14 74HCT04N, IC15 74HC151N, IC16 74HC151N, IC17 74HCT32N, IC18 74HCT374N, IC19 74ACT02N, IC2 74HCT08N, IC20 74HCT08N, IC21 74ACT157N, IC22 74HC151N, IC23 74HC151N, IC24 74HCT08N, IC25 74AC86N, IC26 74HCT374N, IC27 74ACT157N, IC28 74AC08N, IC29 74ACT02N, IC3 74HC151N, IC30 74HCT08N, IC31 74HC151N, IC32 74HC151N, IC33 74HCT374N, IC34 74ACT157N, IC35 74HC373N, IC36 74HC373N, IC37 74HC151N, IC38 74HC151N, IC39 74ACT02N, IC4 74HC151N, IC40 74HCT08N, IC41 74HCT374N, IC42 74HC151N, IC43 74HC151N, IC44 74ACT02N, IC45 74HCT374N, IC46 74HC151N, IC47 74HC151N, IC48 74HCT32N, IC49 74HCT32N, IC5 74HCT374N, IC50 74HC151N, IC51 74HC151N, IC52 74HCT08N, IC53 74HC74N, IC54 74HC74N, IC55 74HCT32N, IC56 74HCT32N, IC57 74HC193N, IC58 74HC193N, IC59 74HCT08N, IC6 74AC08N, IC60 74HC193N, IC62 74HCT08N, IC64 74HC193N, IC65 74HCT32N, IC66 74HCT374N, IC67 74HCT04N, IC68 74HCT32N, IC69 74HC193N, IC7 74AC08N, IC70 74HCT32N, IC71 74HCT32N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

Commit message: add STR and LDR varianst with auto-postincrement.
remove PTR_ADD instruction. usually increment by 1 is enough for most needs.
Parts:
- added IC61: 74HCT08N, 74xx-eu:74HCT08N
Connections:
- removed net ALU_OUTPUT_ENABLE/FILL_PTR_L_PTR_ADD: IC55A.I1, IC62B.I1, IC62D.I1, IC72B.O
- removed net LATCH_ALU_INPUT_B/WRITE_REGB_TO_DBUS_PTR_ADD: IC1C.I1, IC89A.O
- removed net N$166: IC108C.I0, IC59C.I0, IC71B.O
- removed net N$47: IC12A.!A!/B, IC17A.O
- removed net STORE_ALU_OUTPUT/STORE_CARRY_TMP_PTR_ADD: IC112C.I1, IC52A.O
- removed net WRITE_PTR_L_TO_DBUS_PTR_ADD: IC12A.1B, IC17A.I1, IC99B.O
- new net LDR_I: IC89A.I1, IC91C.O, IC99B.I1
- new net N$100: IC92A.I0
- new net N$101: IC88C.I0
- new net N$108: IC89A.O
- new net N$17: IC59B.I1, IC92C.I0
- new net N$32: IC61C.I1, IC95A.O
- new net N$33: IC78C.I0
- new net N$79: IC99A.I0
- new net N$90: IC61C.O
- new net N$91: IC100A.I0
- new net N$92: IC92B.I0
- new net N$93: IC126A.I0
- new net N$94: IC126D.I0
- new net N$95: IC126C.I0
- new net N$96: IC99B.I0
- new net N$98: IC99B.O
- new net N$99: IC89A.I0
- net CARRY&&!IR_DATA: no longer IC62B.I0
- net CARRY&&IR_DATA: no longer IC62D.I0
- net LDR: now also IC91D.O; no longer IC95A.O
- net N$97: now also IC91B.O; no longer IC91C.O
- net PTR_ADD: no longer IC52A.I1, IC71B.I1, IC72B.I1, IC89A.I1, IC91B.O, IC99B.I1
- net PTR_HIGH_COUNT_DOWN: no longer IC62D.O
- net PTR_HIGH_COUNT_UP: no longer IC62B.O
- net SAVE_LR/RET: no longer IC59B.I1, IC91D.O, IC92C.I0
- net SECOND_LATCH_SELECT: now also IC12A.!A!/B; no longer IC17A.I0
- net STATE_0/CYCL_3: now also IC61C.I0; no longer IC78C.I0, IC99A.I0, IC99B.I0
- net STATE_1/CYCL_4: no longer IC100A.I0, IC89A.I0, IC92A.I0, IC92B.I0
- net STATE_2/CYCL_5: no longer IC126A.I0, IC126D.I0, IC52A.I0, IC88C.I0
- net STATE_3/CYCL_6: no longer IC126C.I0, IC72B.I0
- net STORE_ALU_OUTPUT/STORE_CARRY_TMP_JMP_O: now also IC67E.I; no longer IC112C.I0
- net STORE_ALU_OUTPUT_JMP_PTR_ADD: no longer IC112C.O, IC67E.I
- net WQWJKDHSAAASDFXGHCJFDSAAS: now also IC108C.I0, IC59C.I0; no longer IC71B.I0
Other:
- note added: "LDR_I"
- note added: "STR_I"
- note removed: "PTR_ADD"
- moved on the sheet: IC100A, IC100C, IC108C, IC126A, IC126C, IC126D, IC59B, IC59C, IC78C, IC88C, IC89A, IC92A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

Commit message: feature freeze. I will now solder the Control Unit
Parts:
- removed C1, C10, C100, C101, C102, C103, C104, C105, C106, C107, C108, C11, C12, C13, C14, C15, C16, C17, C18, C19, C2, C20, C21, C22, C23, C24, C25, C26, C27, C28, C29, C3, C30, C31, C32, C33, C34, C35, C36, C37, C38, C39, C4, C40, C41, C42, C43, C44, C45, C46, C47, C48, C49, C5, C50, C51, C52, C53, C54, C55, C56, C57, C58, C59, C6, C60, C61, C62, C63, C64, C65, C66, C67, C68, C69, C7, C70, C71, C72, C73, C74, C75, C76, C77, C78, C79, C8, C80, C81, C82, C83, C84, C85, C86, C87, C88, C89, C9, C90, C91, C92, C93, C94, C95, C96, C97, C98, C99: (no value), rcl:C-EUC1206
- removed IC118: 74HC74N, 74xx-eu:74HC74N
- removed IC62: 74HCT08N, 74xx-eu:74HCT08N
- removed IC66: 74HCT374N, 74xx-eu:74HCT374N
- added IC63: 74HCT08N, 74xx-eu:74HCT08N
- IC17: value 74HCT32N -> 74HC193N; device 74xx-eu:74HCT32N -> custom_parts:74HC193N
- IC61: value 74HCT08N -> 74HC193N; device 74xx-eu:74HCT08N -> custom_parts:74HC193N
Connections:
- net ALU_NR1_ENABLE_JMP_O_PTR_ADD renamed ALU_NR1_ENABLE_JMP_O
- net ALU_NR2_ENABLE_JMP_O_PTR_ADD renamed ALU_NR2_ENABLE_JMP_O
- removed net CARRY_LAST_CYCLE: IC118B.Q, IC62A.I0, IC62C.I1
- removed net FILL_LR_H_SAVE_LR: IC126D.O, IC44D.I0
- removed net INPUT_REG2: IC10A.I0, IC10B.I0, IC28C.O, IC30C.I0, IC9A.3B
- removed net LATCH_ALU_INPUT_ALU/JMP_O/PTR_ADD: IC103A.ENC, IC1B.I0, IC1C.O
- removed net N$100: IC92A.I0
- removed net N$101: IC88C.I0
- removed net N$108: IC89A.O
- removed net N$220: IC48B.O, IC48C.I0
- removed net N$230: IC48A.I0, IC48D.O
- removed net N$32: IC61C.I1, IC95A.O
- removed net N$81: IC129D.O, IC129E.I
- removed net N$83: IC129E.O, IC129F.I
- removed net N$84: IC129F.O, IC130A.I1
- removed net N$86: IC112B.O, IC55A.I0
- removed net N$90: IC61C.O
- removed net N$91: IC100A.I0
- removed net N$92: IC92B.I0
- removed net N$95: IC126C.I0
- removed net N$96: IC99B.I0
- removed net N$98: IC99B.O
- removed net N$99: IC89A.I0
- removed net OPC_67_OUPUT2: IC20C.I0, IC6C.I1, IC7C.O
- removed net OPC_67_OUPUT3: IC20D.I0, IC6D.I1, IC7D.O
- removed net POP: IC100B.I1, IC130D.I1, IC48A.I1, IC95D.O
- removed net PTR_ADD: IC48B.I1
- removed net PTR_HIGH_COUNT_DOWN: IC69A.DN
- removed net PTR_HIGH_COUNT_UP: IC69A.UP
- removed net SAVE_LR/RET: IC48D.I1
- removed net STORE_ALU_OUTPUT/STORE_CARRY_TMP_JMP_O: IC40D.O, IC67E.I
- removed net STORE_ALU_OUTPUT_JMP_PTR_ADD: IC112D.I1
- new net FILL_LR_H/COUNT_PC_DOWN_SAVE_LR: IC126D.O, IC129D.I, IC44D.I0
- new net INPUT_REG2/OPC_4/5==11: IC10A.I0, IC10B.I0, IC28C.O, IC30C.I0, IC63B.I0, IC63D.I0, IC9A.3B
- new net LATCH_ALU_INPUT_ALU_JMP_O: IC103A.ENC, IC1A.O, IC1B.I0
- new net LDR/LDR_I: IC100C.I1, IC1C.O, IC48A.I0
- new net N$109: IC19D.O, IC63A.I1
- new net OPC==E: IC19D.I1, IC63D.O, IC92C.I1
- new net OPC==F: IC19D.I0, IC59B.I0, IC63B.O
- new net OPC_67_OUPUT2==11: IC20C.I0, IC63B.I1, IC6C.I1, IC7C.O
- new net OPC_67_OUPUT3==10: IC20D.I0, IC63D.I1, IC6D.I1, IC7D.O
- new net PC_COUNT_UP_SAVE_LR: IC48B.I1, IC52A.O
- new net POP/SAVE_LR/RET: IC48A.I1, IC59B.I1, IC63A.I0, IC92C.I0, IC95D.O
- new net PTR_COUNT_UP: IC129F.O, IC17A.UP
- new net PTR_COUNT_UP_LDR_I: IC55A.I0, IC89A.O
- new net PTR_COUNT_UP_STR_I: IC55A.I1, IC99B.O
- new net STORE_ALU_OUTPUT_JMP_O: IC40D.O, IC49B.I1, IC88B.I1, IC88D.I1
- new net STR/STR_I: IC100D.I1, IC130C.I1, IC48C.I0, IC71A.O
- new net STR_I: IC71A.I0, IC95A.O, IC99B.I1
- net !CLR_CARRY_BIT: now also IC131A.CLR; no longer IC118A.CLR
- net !ENABLE_REG_OUTPUT: now also IC112B.I1, IC112D.O; no longer IC55D.O, IC65B.I1
- net !IR_DATA_OUT_7: now also IC99C.I1; no longer IC62A.I1
- net !OPCODE_5: no longer IC92C.I1
- net !REGISTER_RESET: now also IC17A.CLR, IC61A.CLR
- net !SET_CARRY_BIT: now also IC131A.PRE; no longer IC118A.PRE
- net ALU_CARRY_BIT: now also IC131A.Q; no longer IC118A.Q
- net ALU_CARRY_OUT: now also IC131A.D, IC72B.I1, IC99C.I0; no longer IC118A.D, IC118B.D
- net ALU_OUTPUT_ENABLE/FILL_PC_L_JMP_O: now also IC49A.I1; no longer IC112B.I1, IC88B.I1, IC88D.I1
- net CARRY&&!IR_DATA: now also IC99C.O; no longer IC62A.O
- net CARRY&&IR_DATA: now also IC72B.O; no longer IC62C.O
- net CLR_NOT_OE/CLR_NOT_CS/PC_COUNT_UP_CYCL_2: now also IC55D.I0; no longer IC49A.I0
- net CYCLE1/CYLCE2: now also IC68B.I0; no longer IC71A.I0
- net DATA0: now also IC17A.A; no longer IC66A.1D
- net DATA1: now also IC17A.B; no longer IC66A.2D
- net DATA2: now also IC17A.C; no longer IC66A.3D
- net DATA3: now also IC17A.D; no longer IC66A.4D
- net DATA4: now also IC61A.A; no longer IC66A.5D
- net DATA5: now also IC61A.B; no longer IC66A.6D
- net DATA6: now also IC61A.C; no longer IC66A.7D
- net DATA7: now also IC61A.D; no longer IC66A.8D
- net DBUS_SELECTOR_TABLE_2: now also IC55C.O; no longer IC17C.O
- net ENABLE_ALU_OUTPUT: now also IC112D.I1, IC49A.O, IC67E.I; no longer IC14D.I, IC55A.O, IC55D.I1
- net ENABLE_ALU_OUTPUT/FILL_REGISTER_ALU: now also IC112C.I1, IC49A.I0; no longer IC112B.I0, IC17D.I1
- net FILL_PC_L/WRITE_LR_H_DBUS_RET: now also IC65B.I0; no longer IC49B.I0
- net FILL_REGISTER_MOV: now also IC112C.I0; no longer IC17D.I0
- net GND: now also IC12A.1B; no longer C1.2, C10.2, C100.2, C101.2, C102.2, C103.2, C104.2, C105.2, C106.2, C107.2, C108.2, C11.2, C12.2, C13.2, C14.2, C15.2, C16.2, C17.2, C18.2, C19.2, C2.2, C20.2, C21.2, C22.2, C23.2, C24.2, C25.2, C26.2, C27.2, C28.2, C29.2, C3.2, C30.2, C31.2, C32.2, C33.2, C34.2, C35.2, C36.2, C37.2, C38.2, C39.2, C4.2, C40.2, C41.2, C42.2, C43.2, C44.2, C45.2, C46.2, C47.2, C48.2, C49.2, C5.2, C50.2, C51.2, C52.2, C53.2, C54.2, C55.2, C56.2, C57.2, C58.2, C59.2, C6.2, C60.2, C61.2, C62.2, C63.2, C64.2, C65.2, C66.2, C67.2, C68.2, C69.2, C7.2, C70.2, C71.2, C72.2, C73.2, C74.2, C75.2, C76.2, C77.2, C78.2, C79.2, C8.2, C80.2, C81.2, C82.2, C83.2, C84.2, C85.2, C86.2, C87.2, C88.2, C89.2, C9.2, C90.2, C91.2, C92.2, C93.2, C94.2, C95.2, C96.2, C97.2, C98.2, C99.2, IC66A.OC, JP4.36
- net INPUT_REG_IS_NOT_OUTPUT_REG: now also IC71B.O; no longer IC17B.O
- net IR_DATA_OUT_7: now also IC72B.I0; no longer IC62C.I0
- net LDR: now also IC1C.I1; no longer IC100C.I1, IC48D.I0
- net LDR_I: now also IC1C.I0; no longer IC99B.I1
- net MEM_OE: now also IC112D.I0, IC68B.O; no longer IC55D.I0, IC71A.O
- net N$11: now also IC129F.I, IC55A.O; no longer IC1A.O, IC1C.I0
- net N$13: now also IC48D.O; no longer IC68B.O
- net N$14: now also IC39D.I1, IC48B.O; no longer IC118B.CLK, IC67E.O
- net N$17: now also IC100B.I1, IC130D.I1, IC63A.O; no longer IC59B.I1, IC92C.I0
- net N$171: now also IC65B.O; no longer IC49B.O
- net N$194: now also IC52A.I1
- net N$2: now also IC129E.I; no longer IC67D.I
- net N$203: now also IC129E.O; no longer IC67D.O
- net N$21: now also IC48D.I1; no longer IC68B.I1
- net N$33: now also IC17A.BO, IC61A.DN; no longer IC78C.I0
- net N$48: now also IC71B.I0; no longer IC17B.I0
- net N$5: now also IC55D.I1; no longer IC49A.I1
- net N$51: now also IC71B.I1; no longer IC17B.I1
- net N$52: now also IC131B.CLK; no longer IC129D.I, IC130A.I0
- net N$56: now also IC55D.O; no longer IC49A.O
- net N$6: now also IC112C.O; no longer IC17D.O
- net N$74: now also IC131A.CLK, IC67D.O; no longer IC118A.CLK, IC129A.O
- net N$79: now also IC17A.CO, IC61A.UP; no longer IC99A.I0
- net N$80: now also IC48D.I0; no longer IC68B.I0
- net N$85: now also IC112B.I0; no longer IC65B.I0
- net N$87: now also IC129D.O, IC57A.DN; no longer IC130A.O, IC131B.CLK
- net N$89: now also IC67E.O; no longer IC14D.O
- net N$93: now also IC61A.BO, IC69A.DN; no longer IC126A.I0
- net N$94: now also IC61A.CO, IC69A.UP; no longer IC126D.I0
- net OPCODE_5: no longer IC59B.I0
- net PC_COUNT_UP_RET: now also IC48B.I0; no longer IC39D.I1
- net PC_L_TO_DBUS: now also IC65B.I1; no longer IC49B.I1
- net PTR_DATA_OUT_0: now also IC17A.QA; no longer IC66A.1Q
- net PTR_DATA_OUT_1: now also IC17A.QB; no longer IC66A.2Q
- net PTR_DATA_OUT_2: now also IC17A.QC; no longer IC66A.3Q
- net PTR_DATA_OUT_3: now also IC17A.QD; no longer IC66A.4Q
- net PTR_DATA_OUT_4: now also IC61A.QA; no longer IC66A.5Q
- net PTR_DATA_OUT_5: now also IC61A.QB; no longer IC66A.6Q
- net PTR_DATA_OUT_6: now also IC61A.QC; no longer IC66A.7Q
- net PTR_DATA_OUT_7: now also IC61A.QD; no longer IC66A.8Q
- net PTR_L_LOAD_INPUT_NOT: now also IC17A.LD, IC61A.LD; no longer IC66A.CLK
- net REGS_OUTPUT_TO_DATABUS_ENABLE: now also IC112B.O; no longer IC65B.O
- net SP_COUNT_UP/WRITE_REG_TO_DBUS_SELECTOR2_PUSH: now also IC55C.I1; no longer IC17C.I1
- net STATE_0/CYCL_3: now also IC52A.I0, IC99A.I0; no longer IC61C.I0
- net STATE_1/CYCL_4: now also IC100A.I0, IC78C.I0, IC89A.I0, IC92A.I0
- net STATE_2/CYCL_5: now also IC126A.I0, IC88C.I0, IC92B.I0, IC99B.I0
- net STATE_3/CYCL_6: now also IC126C.I0, IC126D.I0, JP4.36
- net STORE_ALU_OUTPUT: now also IC49B.O; no longer IC112D.O
- net STORE_ALU_OUTPUT/STORE_CARRY_ALU: now also IC49B.I0, IC67D.I; no longer IC112D.I0, IC129A.I
- net STR: now also IC71A.I1; no longer IC100D.I1, IC130C.I1, IC48B.I0
- net VCC: now also IC17A.DN; no longer C1.1, C10.1, C100.1, C101.1, C102.1, C103.1, C104.1, C105.1, C106.1, C107.1, C108.1, C11.1, C12.1, C13.1, C14.1, C15.1, C16.1, C17.1, C18.1, C19.1, C2.1, C20.1, C21.1, C22.1, C23.1, C24.1, C25.1, C26.1, C27.1, C28.1, C29.1, C3.1, C30.1, C31.1, C32.1, C33.1, C34.1, C35.1, C36.1, C37.1, C38.1, C39.1, C4.1, C40.1, C41.1, C42.1, C43.1, C44.1, C45.1, C46.1, C47.1, C48.1, C49.1, C5.1, C50.1, C51.1, C52.1, C53.1, C54.1, C55.1, C56.1, C57.1, C58.1, C59.1, C6.1, C60.1, C61.1, C62.1, C63.1, C64.1, C65.1, C66.1, C67.1, C68.1, C69.1, C7.1, C70.1, C71.1, C72.1, C73.1, C74.1, C75.1, C76.1, C77.1, C78.1, C79.1, C8.1, C80.1, C81.1, C82.1, C83.1, C84.1, C85.1, C86.1, C87.1, C88.1, C89.1, C9.1, C90.1, C91.1, C92.1, C93.1, C94.1, C95.1, C96.1, C97.1, C98.1, C99.1, IC118B.CLR, IC118B.PRE, IC57A.DN
- net WRITE_PTR_TO_ABUS/CLR_NOT_OE/CLR_NOT_CS/FILL_REGISTER_LDR: now also IC68B.I1; no longer IC71A.I1
- net WRITE_REG_TO_DBUS_SELECTOR2_STR: now also IC55C.I0; no longer IC17C.I0
Other:
- note added: "CYCL_3"
- note added: "Write reg to dbus every cycle"
- note added: "count down because SAVE_LR counts up in Cycle1 and down in Cycle5"
- note removed: "Activate MOV signal only when REG0(MOVZ) is zero"
- note removed: "InstructionRegister_LOW"
- note removed: "Needs to count up twice actually"
- note removed: "PC only counts up"
- note removed: "Write reg to dbus in every cycle"
- moved on the sheet: IC100A, IC100B, IC100D, IC101, IC103, IC105A, IC11, IC112A, IC112B, IC112D, IC126A, IC126B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
