File: schematics/UI_board/ui_board.sch (EAGLE design)
At the start: 52 parts, among them IC1 74HCT00N, IC10 74HCT32N, IC11 74HCT14N, IC12 74HCT14N, IC2 74HCT151N, IC3 74HCT174N, IC4 74HCT74N, IC5 74HCT04N, IC6 74HCT08N, IC7 74HC148N, IC8 74HCT373N, IC9 74HCT32N

Commit message: changed register chips to 74xx374
Parts:
- added C10, C11, C12, C13: 1µF, rcl:C-EU025-024X044
- added IC13: 74HCT14N, 74xx-eu:74HCT14N
- added R21, R23, R25, R27: 10k, rcl:R-EU_0204/7
- added R22, R24, R26, R28: 22k, rcl:R-EU_0204/7
- added S11, S12, S13, S14: (no value), switch-omron:10-XX
Connections:
- removed net N$17: IC7A.EI
- new net CHANGE_CLOCK_SELECT10: IC12E.O, IC5D.I
- new net CHANGE_CLOCK_SELECT11: IC13C.O, IC5E.I
- new net CHANGE_CLOCK_SELECT4: IC12C.O, IC5B.I
- new net CHANGE_CLOCK_SELECT9: IC12D.O, IC5C.I
- new net N$48: R23.1, R24.1, S12.S, S12.S1
- new net N$50: R21.1, R22.1, S11.S, S11.S1
- new net N$51: C10.1, IC12C.I, R22.2
- new net N$52: C11.1, IC12D.I, R24.2
- new net N$53: R25.1, R26.1, S13.S, S13.S1
- new net N$54: C12.1, IC12E.I, R26.2
- new net N$55: R27.1, R28.1, S14.S, S14.S1
- new net N$56: C13.1, IC13C.I, R28.2
- net !CLR_CARRY_BIT: now also IC5D.O
- net !REGISTER_RESET: now also IC5B.O
- net !RING_CNTR_RESET: now also IC5C.O
- net !SET_CARRY_BIT: now also IC5E.O
- net GND: now also C10.2, C11.2, C12.2, C13.2, IC7A.EI, S11.P, S11.P1, S12.P, S12.P1, S13.P, S13.P1, S14.P, S14.P1
- net VCC: now also R21.2, R23.2, R25.2, R27.2
Other:
- moved on the sheet: IC12C, IC12D, IC12E, IC1A, IC1C, JP1, R1, R2, S1

Commit message: start ui board layout
Parts:
- removed C1: 1µF, rcl:C-EU025-024X044
- removed R3: 10k, rcl:R-EU_0204/7
- removed R4: 22k, rcl:R-EU_0204/7
- removed S2: (no value), switch-omron:10-XX
- added C14: 1µF, rcl:C-EU025-024X044
- added IC14: 74HCT14N, 74xx-eu:74HCT14N
- added JP2: (no value), pinhead:PINHD-1X8
- added JP3: (no value), pinhead:PINHD-1X2
- added LED1, LED10, LED11, LED12, LED13, LED14, LED15, LED16, LED17, LED18, LED19, LED2, LED20, LED3, LED4, LED5, LED6, LED7, LED8, LED9: (no value), led:LED3MM
- added QG2: (no value), crystal:XO-14
- added R29, R30, R31, R32, R33, R34, R35, R36, R37, R38, R39, R40, R41, R42, R43, R44, R45, R46, R47, R48, R52: 22k, rcl:R-EU_R1206
- added R51: 10k, rcl:R-EU_R1206
- added S16: (no value), switch-omron:10-XX
- IC13: value 74HCT14N -> 74HCT393N; device 74xx-eu:74HCT14N -> 74xx-eu:74HCT393N
- R1, R2: device rcl:R-EU_0207/10 -> rcl:R-EU_R1206
- R10, R11, R12, R13, R14, R15, R16, R17, R18, R19, R20, R21, R22, R23, R24, R25, R26, R27, R28, R5, R6, R7, R8, R9: device rcl:R-EU_0204/7 -> rcl:R-EU_R1206
Connections:
- removed net 100KHZ: IC2A.D2
- removed net 10HZ: IC2A.D1
- removed net 12MHZ: IC2A.D7
- removed net N$32: IC8A.ENC, IC9A.O
- removed net N$33: R3.1, R4.1, S2.S, S2.S1
- removed net N$34: C1.1, IC12F.I, R4.2
- new net 31.25KHZ: IC13B.QD, IC2A.D1
- new net 500KHZ: IC13A.QD, IC13B.A, IC2A.D2
- new net N$17: LED20.C, R38.1
- new net N$57: LED10.C, R39.2
- new net N$58: LED12.C, R40.2
- new net N$59: LED13.C, R41.2
- new net N$60: LED2.C, R29.2
- new net N$61: LED1.C, R30.2
- new net N$62: LED3.C, R31.2
- new net N$63: LED4.C, R32.2
- new net N$64: LED5.C, R33.2
- new net N$65: LED6.C, R34.2
- new net N$66: LED7.C, R35.2
- new net N$67: LED8.C, R36.2
- new net N$68: LED9.C, R37.2
- new net N$69: LED14.C, R42.2
- new net N$70: LED15.C, R43.2
- new net N$71: LED16.C, R44.2
- new net N$72: LED17.C, R45.2
- new net N$73: LED18.C, R46.2
- new net N$74: LED19.C, R47.1
- new net N$75: LED11.C, R48.1
- new net N$79: R51.1, R52.1, S16.S, S16.S1
- new net N$80: C14.1, IC12F.I, R52.2
- net !RESET_CLOCK_SELECT: now also IC12F.O
- net 1MHZ: now also IC13A.QC
- net 2MHZ: now also IC13A.QB
- net 4MHZ: now also IC13A.QA
- net 8MHZ: now also IC13A.A, QG2.OUT
- net ALU_CARRY_BIT: now also LED11.A
- net CHANGE_CLOCK_SELECT: now also IC8A.ENC, IC9A.O; no longer IC12F.O
- net CHANGE_CLOCK_SELECT11: now also IC14B.O; no longer IC13C.O
- net CYCL_1: now also LED2.A
- net CYCL_2: now also LED1.A
- net CYCL_3: now also LED3.A
- net CYCL_4: now also LED4.A
- net CYCL_5: now also LED5.A
- net CYCL_6: now also LED6.A
- net CYCL_7: now also LED7.A
- net CYCL_8: now also LED8.A
- net CYCL_9: now also LED9.A
- net GND: now also C14.2, IC13A.CLR, IC13B.CLR, IC2A.D7, JP3.1, QG2.GND, R29.1, R30.1, R31.1, R32.1, R33.1, R34.1, R35.1, R36.1, R37.1, R38.2, R39.1, R40.1, R41.1, R42.1, R43.1, R44.1, R45.1, R46.1, R47.2, R48.2, S16.P, S16.P1; no longer C1.2, S2.P, S2.P1
- net N$18: now also JP2.1
- net N$19: now also JP2.2
- net N$20: now also JP2.3
- net N$21: now also JP2.4
- net N$22: now also JP2.5
- net N$23: now also JP2.6
- net N$24: now also JP2.7
- net N$25: now also JP2.8
- net N$56: now also IC14B.I; no longer IC13C.I
- net REG0_OUT_0: now also LED10.A
- net REG0_OUT_1: now also LED12.A
- net REG0_OUT_2: now also LED13.A
- net REG0_OUT_3: now also LED14.A
- net REG0_OUT_4: now also LED15.A
- net REG0_OUT_5: now also LED16.A
- net REG0_OUT_6: now also LED17.A
- net REG0_OUT_7: now also LED18.A
- net REG0_ZERO: now also LED20.A
- net SP_DATA_OVER/UNDERFLOW: now also LED19.A
- net VCC: now also QG2.VCC, R51.2; no longer R3.2
Other:
- note added: "maybe need some time delay here"
- moved on the sheet: C10, C12, C13, C2, C3, C4, C5, C6, C7, C8, C9, IC10B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

Commit message: fix. gonna try to reduce cycles to 8 per instruction now
Parts:
- removed IC14: 74HCT14N, 74xx-eu:74HCT14N
- removed IC7: 74HC148N, 74xx-eu:74HC148N
- removed R27, R51: 10k, rcl:R-EU_R1206
- removed R28, R52: 22k, rcl:R-EU_R1206
- removed S14, S16: (no value), switch-omron:10-XX
- added C1: 1µF, rcl:C-EU025-024X044
- added C15, C16, C17, C18, C19, C20, C21, C22, C23: (no value), rcl:C-EUC1206
- added JP4: (no value), pinhead:PINHD-2X5
- added R3: 10k, rcl:R-EU_R1206
- added R4: 22k, rcl:R-EU_R1206
- added S2: (no value), switch-omron:10-XX
- C13, C14: value 1µF -> (none); device rcl:C-EU025-024X044 -> rcl:C-EUC1206
- IC3: value 74HCT174N -> 74HCT32N; device 74xx-eu:74HCT174N -> 74xx-eu:74HCT32N
- IC6: value 74HCT08N -> 74HCT32N; device 74xx-eu:74HCT08N -> 74xx-eu:74HCT32N
Connections:
- removed net !RESET_CLOCK_SELECT: IC12F.O, IC3A.CLR
- removed net CHANGE_CLOCK_SELECT10: IC12E.O, IC5D.I
- removed net CHANGE_CLOCK_SELECT11: IC14B.O, IC5E.I
- removed net CHANGE_CLOCK_SELECT4: IC12C.O, IC5B.I
- removed net CHANGE_CLOCK_SELECT9: IC12D.O, IC5C.I
- removed net N$54 (its old number): C12.1, IC12E.I, R26.2
- removed net N$56: C13.1, IC14B.I, R28.2
- removed net N$79: R51.1, R52.1, S16.S, S16.S1
- removed net N$80: C14.1, IC12F.I, R52.2
- new net N$32: IC3C.O, IC6C.I1
- new net N$33: IC3A.O, IC6B.I0
- new net N$34: IC6A.O, IC6B.I1
- new net N$48: C1.1, IC12E.I, R4.2
- new net N$76: IC3B.I0, IC8A.3Q, JP2.3
- new net TIMER_CLOCK: JP1.3, JP4.10, JP4.2, JP4.4, JP4.6, JP4.8
- net !CLR_CARRY_BIT: now also IC12D.O; no longer IC5D.O
- net !REGISTER_RESET: now also IC12F.O; no longer IC5B.O
- net !RING_CNTR_RESET: now also IC12E.O; no longer IC5C.O
- net !SET_CARRY_BIT: now also IC12C.O; no longer IC5E.O
- net 1MHZ: now also JP4.5
- net 2MHZ: now also JP4.3
- net 31.25KHZ: now also JP4.9
- net 4MHZ: now also JP4.1
- net 500KHZ: now also JP4.7
- net ALU_CARRY_BIT: now also JP1.16; no longer JP1.7
- net CHANGE_CLOCK_SELECT: now also IC1D.I1; no longer IC3A.CLK, IC6A.I1
- net GND: now also C15.2, C16.2, C17.2, C18.2, C19.2, C20.2, C21.2, C22.2, C23.2, IC8A.OC, JP1.11, JP1.13, JP1.7, JP1.9, R21.2, R23.2, R25.2, R3.2; no longer C10.2, C11.2, C12.2, IC7A.EI, JP1.16, JP1.18, JP1.20, JP1.3, S11.P, S11.P1, S12.P, S12.P1, S13.P, S13.P1, S14.P, S14.P1, S16.P, S16.P1
- net N$1: now also IC1B.I0; no longer IC6B.I0
- net N$10: now also IC5F.O; no longer IC6A.O
- net N$11: now also IC2A.A, IC6C.O; no longer IC3A.D1, IC7A.A0
- net N$12: now also IC3D.O, IC6C.I0, IC6D.I0; no longer IC3A.D2, IC7A.A1
- net N$13: now also IC2A.C, IC6B.O; no longer IC3A.D3, IC7A.A2
- net N$18: now also IC3B.O, IC6D.I1; no longer IC7A.0, IC8A.1Q, JP2.1
- net N$19: now also IC3C.I1; no longer IC7A.1
- net N$20: now also R3.1, R4.1, S2.S, S2.S1; no longer IC7A.2, IC8A.3Q, JP2.3
- net N$21: now also IC3D.I1; no longer IC7A.3
- net N$22: now also IC3A.I0; no longer IC7A.4
- net N$23: now also IC3A.I1, IC3C.I0; no longer IC7A.5
- net N$24: now also IC3B.I1, IC6A.I0; no longer IC7A.6
- net N$25: now also IC3D.I0, IC6A.I1; no longer IC7A.7
- net N$4: now also IC1D.O, IC5F.I; no longer IC2A.A, IC3A.Q1
- net N$51: now also IC12F.I; no longer IC12C.I
- net N$55: now also C12.1, IC12C.I, R26.2; no longer R27.1, R28.1, S14.S, S14.S1
- net N$6: now also IC6D.O; no longer IC3A.Q2
- net N$7: now also IC8A.1Q, JP2.1; no longer IC2A.C, IC3A.Q3
- net N$8: now also IC1D.I0; no longer IC6A.I0
- net REG0_ZERO: now also JP1.20; no longer JP1.11
- net RING_CNTR_CLOCK: now also IC1B.O; no longer IC6B.O
- net SELECTED_CLOCK: now also IC1B.I1; no longer IC6B.I1
- net SP_DATA_OVER/UNDERFLOW: now also JP1.18; no longer JP1.9
- net VCC: now also C1.2, C10.2, C11.2, C12.2, C13.1, C14.1, C15.1, C16.1, C17.1, C18.1, C19.1, C20.1, C21.1, C22.1, C23.1, JP3.2, S11.P, S11.P1, S12.P, S12.P1, S13.P, S13.P1, S2.P, S2.P1; no longer R21.2, R23.2, R25.2, R27.2, R51.2
Other:
- moved on the sheet: C10, C11, C12, C13, C14, IC12C, IC12D, IC12E, IC12F, IC13A, IC13B, IC1A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
