File: schematics/UI_board/ui_board.sch (EAGLE design)
At the start: 114 parts, among them IC1 74HCT00N, IC10 74HCT32N, IC11 74HCT14N, IC12 74HCT14N, IC13 74HCT393N, IC2 74HCT151N, IC3 74HCT32N, IC4 74HCT74N, IC5 74HCT04N, IC6 74HCT32N, IC8 74HCT373N, IC9 74HCT32N

Commit message: clean up docs and schematic. no functional changes
Other:
- moved on the sheet: IC13B, IC1D, IC5F, QG2
Changed lines of the file:
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@@
 <instance part="LED19" gate="G$1" x="-12.7" y="-33.02" rot="MR90"/>
 <instance part="LED20" gate="G$1" x="-12.7" y="-40.64" rot="MR90"/>
-<instance part="QG2" gate="G$1" x="38.1" y="266.7"/>
+<instance part="QG2" gate="G$1" x="43.18" y="266.7"/>
 <instance part="JP2" gate="A" x="-17.78" y="193.04"/>
 <instance part="IC13" gate="A" x="81.28" y="264.16"/>
-<instance part="P+3" gate="VCC" x="22.86" y="279.4"/>
-<instance part="GND5" gate="1" x="22.86" y="254"/>
+<instance part="P+3" gate="VCC" x="27.94" y="279.4"/>
+<instance part="GND5" gate="1" x="27.94" y="254"/>
 <instance part="GND6" gate="1" x="66.04" y="254"/>
-<instance part="IC13" gate="B" x="121.92" y="246.38"/>
-<instance part="GND35" gate="1" x="106.68" y="236.22"/>
+<instance part="IC13" gate="B" x="124.46" y="246.38"/>
+<instance part="GND35" gate="1" x="109.22" y="236.22"/>
 <instance part="JP3" gate="G$1" x="10.16" y="104.14" rot="R180"/>
 <instance part="GND38" gate="1" x="17.78" y="91.44"/>
@@
 <instance part="GND36" gate="1" x="-63.5" y="175.26"/>
 <instance part="IC1" gate="B" x="167.64" y="157.48"/>
-<instance part="IC1" gate="D" x="142.24" y="177.8"/>
-<instance part="IC5" gate="F" x="165.1" y="177.8"/>
+<instance part="IC1" gate="D" x="142.24" y="180.34"/>
+<instance part="IC5" gate="F" x="165.1" y="180.34"/>
 <instance part="JP4" gate="A" x="160.02" y="261.62"/>
 <instance part="IC3" gate="D" x="7.62" y="213.36"/>
@@
 <segment>
 <pinref part="QG2" gate="G$1" pin="VCC"/>
-<wire x1="25.4" y1="271.78" x2="22.86" y2="271.78" width="0.1524" layer="91"/>
-<wire x1="22.86" y1="271.78" x2="22.86" y2="276.86" width="0.1524" layer="91"/>
+<wire x1="30.48" y1="271.78" x2="27.94" y2="271.78" width="0.1524" layer="91"/>
+<wire x1="27.94" y1="271.78" x2="27.94" y2="276.86" width="0.1524" layer="91"/>
 <pinref part="P+3" gate="VCC" pin="VCC"/>
 </segment>
@@
 <segment>
 <pinref part="QG2" gate="G$1" pin="GND"/>
-<wire x1="25.4" y1="261.62" x2="22.86" y2="261.62" width="0.1524" layer="91"/>
-<wire x1="22.86" y1="261.62" x2="22.86" y2="256.54" width="0.1524" layer="91"/>
+<wire x1="30.48" y1="261.62" x2="27.94" y2="261.62" width="0.1524" layer="91"/>
+<wire x1="27.94" y1="261.62" x2="27.94" y2="256.54" width="0.1524" layer="91"/>
 <pinref part="GND5" gate="1" pin="GND"/>
 </segment>
@@
 <segment>
 <pinref part="IC13" gate="B" pin="CLR"/>
-<wire x1="109.22" y1="241.3" x2="106.68" y2="241.3" width="0.1524" layer="91"/>
-<wire x1="106.68" y1="241.3" x2="106.68" y2="238.76" width="0.1524" layer="91"/>
+<wire x1="111.76" y1="241.3" x2="109.22" y2="241.3" width="0.1524" layer="91"/>
+<wire x1="109.22" y1="241.3" x2="109.22" y2="238.76" width="0.1524" layer="91"/>
 <pinref part="GND35" gate="1" pin="GND"/>
 </segment>
@@
 <segment>
 <pinref part="IC13" gate="A" pin="QD"/>
-<wire x1="93.98" y1="259.08" x2="106.68" y2="259.08" width="0.1524" layer="91"/>
+<wire x1="93.98" y1="259.08" x2="109.22" y2="259.08" width="0.1524" layer="91"/>
 <label x="96.52" y="259.08" size="1.778" layer="95"/>
-<wire x1="106.68" y1="259.08" x2="106.68" y2="248.92" width="0.1524" layer="91"/>
+<wire x1="109.22" y1="259.08" x2="109.22" y2="248.92" width="0.1524" layer="91"/>
 <pinref part="IC13" gate="B" pin="A"/>
-<wire x1="106.68" y1="248.92" x2="109.22" y2="248.92" width="0.1524" layer="91"/>
-<junction x="106.68" y="259.08"/>
+<wire x1="109.22" y1="248.92" x2="111.76" y2="248.92" width="0.1524" layer="91"/>
+<junction x="109.22" y="259.08"/>
 <pinref part="JP4" gate="A" pin="7"/>
-<wire x1="106.68" y1="259.08" x2="157.48" y2="259.08" width="0.1524" layer="91"/>
+<wire x1="109.22" y1="259.08" x2="157.48" y2="259.08" width="0.1524" layer="91"/>
 </segment>
 </net>
@@
 <segment>
 <pinref part="QG2" gate="G$1" pin="OUT"/>
-<wire x1="50.8" y1="266.7" x2="66.04" y2="266.7" width="0.1524" layer="91"/>
+<wire x1="55.88" y1="266.7" x2="66.04" y2="266.7" width="0.1524" layer="91"/>
 <pinref part="IC13" gate="A" pin="A"/>
 <wire x1="68.58" y1="266.7" x2="66.04" y2="266.7" width="0.1524" layer="91"/>
@@
 <net name="CHANGE_CLOCK_SELECT" class="0">
 <segment>
-<wire x1="134.62" y1="175.26" x2="129.54" y2="175.26" width="0.1524" layer="91"/>
-<wire x1="129.54" y1="175.26" x2="129.54" y2="152.4" width="0.1524" layer="91"/>
+<wire x1="134.62" y1="177.8" x2="129.54" y2="177.8" width="0.1524" layer="91"/>
+<wire x1="129.54" y1="177.8" x2="129.54" y2="152.4" width="0.1524" layer="91"/>
 <wire x1="129.54" y1="152.4" x2="-58.42" y2="152.4" width="0.1524" layer="91"/>
 <pinref part="IC4" gate="A" pin="D"/>
 <wire x1="187.96" y1="205.74" x2="129.54" y2="205.74" width="0.1524" layer="91"/>
-<wire x1="129.54" y1="205.74" x2="129.54" y2="175.26" width="0.1524" layer="91"/>
-<junction x="129.54" y="175.26"/>
+<wire x1="129.54" y1="205.74" x2="129.54" y2="177.8" width="0.1524" layer="91"/>
+<junction x="129.54" y="177.8"/>
 <pinref part="IC9" gate="A" pin="O"/>
 <wire x1="-60.96" y1="152.4" x2="-58.42" y2="152.4" width="0.1524" layer="91"/>
@@
 <wire x1="218.44" y1="208.28" x2="213.36" y2="208.28" width="0.1524" layer="91"/>
 <pinref part="IC1" gate="D" pin="I0"/>
-<wire x1="134.62" y1="180.34" x2="132.08" y2="180.34" width="0.1524" layer="91"/>
-<wire x1="132.08" y1="180.34" x2="132.08" y2="190.5" width="0.1524" layer="91"/>
+<wire x1="134.62" y1="182.88" x2="132.08" y2="182.88" width="0.1524" layer="91"/>
+<wire x1="132.08" y1="182.88" x2="132.08" y2="190.5" width="0.1524" layer="91"/>
 </segment>
 </net>
@@
 <segment>
 <pinref part="IC4" gate="B" pin="D"/>
-<wire x1="177.8" y1="180.34" x2="187.96" y2="180.34" width="0.1524" layer="91"/>
+<wire x1="175.26" y1="180.34" x2="187.96" y2="180.34" width="0.1524" layer="91"/>
 <pinref part="IC5" gate="F" pin="O"/>
-<wire x1="175.26" y1="177.8" x2="177.8" y2="177.8" width="0.1524" layer="91"/>
-<wire x1="177.8" y1="177.8" x2="177.8" y2="180.34" width="0.1524" layer="91"/>
 </segment>
 </net>
@@
 <segment>
 <pinref part="IC9" gate="D" pin="I0"/>
-<wire x1="-139.7" y1="287.02" x2="-139.7" y2="203.2" width="0.1524" layer="91"/>
-<wire x1="-139.7" y1="203.2" x2="-139.7" y2="175.26" width="0.1524" layer="91"/>
-<wire x1="-139.7" y1="175.26" x2="-116.84" y2="175.26" width="0.1524" layer="91"/>
+<wire x1="-137.16" y1="287.02" x2="-137.16" y2="203.2" width="0.1524" layer="91"/>
+<wire x1="-137.16" y1="203.2" x2="-137.16" y2="175.26" width="0.1524" layer="91"/>
+<wire x1="-137.16" y1="175.26" x2="-116.84" y2="175.26" width="0.1524" layer="91"/>
 <pinref part="IC11" gate="A" pin="O"/>
-<wire x1="-162.56" y1="287.02" x2="-139.7" y2="287.02" width="0.1524" layer="91"/>
+<wire x1="-162.56" y1="287.02" x2="-137.16" y2="287.02" width="0.1524" layer="91"/>
 <pinref part="IC8" gate="A" pin="1D"/>
-<wire x1="-55.88" y1="203.2" x2="-139.7" y2="203.2" width="0.1524" layer="91"/>
-<junction x="-139.7" y="203.2"/>
+<wire x1="-55.88" y1="203.2" x2="-137.16" y2="203.2" width="0.1524" layer="91"/>
+<junction x="-137.16" y="203.2"/>
 </segment>
 </net>
@@
 <net name="CHANGE_CLOCK_SELECT2" class="0">
 <segment>
-<wire x1="-147.32" y1="243.84" x2="-147.32" y2="200.66" width="0.1524" layer="91"/>
+<wire x1="-144.78" y1="243.84" x2="-144.78" y2="200.66" width="0.1524" layer="91"/>
 <pinref part="IC9" gate="D" pin="I1"/>
-<wire x1="-147.32" y1="200.66" x2="-147.32" y2="170.18" width="0.1524" layer="91"/>
-<wire x1="-147.32" y1="170.18" x2="-116.84" y2="170.18" width="0.1524" layer="91"/>
-<wire x1="-162.56" y1="243.84" x2="-147.32" y2="243.84" width="0.1524" layer="91"/>
+<wire x1="-144.78" y1="200.66" x2="-144.78" y2="170.18" width="0.1524" layer="91"/>
+<wire x1="-144.78" y1="170.18" x2="-116.84" y2="170.18" width="0.1524" layer="91"/>
+<wire x1="-162.56" y1="243.84" x2="-144.78" y2="243.84" width="0.1524" layer="91"/>
 <pinref part="IC11" gate="B" pin="O"/>
 <pinref part="IC8" gate="A" pin="2D"/>
-<wire x1="-55.88" y1="200.66" x2="-147.32" y2="200.66" width="0.1524" layer="91"/>
-<junction x="-147.32" y="200.66"/>
+<wire x1="-55.88" y1="200.66" x2="-144.78" y2="200.66" width="0.1524" layer="91"/>
+<junction x="-144.78" y="200.66"/>
 </segment>
 </net>
@@
 <net name="31.25KHZ" class="0">
 <segment>
-<label x="137.16" y="241.3" size="1.778" layer="95"/>
+<label x="139.7" y="241.3" size="1.778" layer="95"/>
 <pinref part="JP4" gate="A" pin="9"/>
-<wire x1="157.48" y1="256.54" x2="149.86" y2="256.54" width="0.1524" layer="91"/>
-<wire x1="149.86" y1="256.54" x2="149.86" y2="241.3" width="0.1524" layer="91"/>
+<wire x1="157.48" y1="256.54" x2="152.4" y2="256.54" width="0.1524" layer="91"/>
+<wire x1="152.4" y1="256.54" x2="152.4" y2="241.3" width="0.1524" layer="91"/>
 <pinref part="IC13" gate="B" pin="QD"/>
-<wire x1="149.86" y1="241.3" x2="134.62" y2="241.3" width="0.1524" layer="91"/>
+<wire x1="152.4" y1="241.3" x2="137.16" y2="241.3" width="0.1524" layer="91"/>
 </segment>
 <segment>
@@
 <pinref part="IC1" gate="D" pin="O"/>
 <pinref part="IC5" gate="F" pin="I"/>
-<wire x1="154.94" y1="177.8" x2="149.86" y2="177.8" width="0.1524" layer="91"/>
-</segment>
-</net>
+<wire x1="154.94" y1="180.34" x2="149.86" y2="180.34" width="0.1524" layer="91"/>
+</segment>
+</net>

Commit message: fix ui_bord. seems to work
Parts:
- removed IC1: 74HCT00N, 74xx-eu:74HCT00N
- removed S1: (no value), switch-omron:10-XX
- added C24: 1µF, rcl:C-EU025-024X044
- added IC7: 74HCT14N, 74xx-eu:74HCT14N
- added R2: 10k, rcl:R-EU_R1206
- added S14: (no value), switch-omron:10-XX
- IC5: value 74HCT04N -> 74HCT08N; device 74xx-eu:74HCT04N -> 74xx-eu:74HCT08N
- R27: value (none) -> 22k
- renumbered R1 to R27
Connections:
- new net N$3: R2.1, R27.1, S14.S, S14.S1
- new net N$56: C24.1, IC7C.I, R27.2
- new net N$67: IC7E.O
- new net N$68: IC5C.I1, IC7A.O
- new net N$77: IC7E.I
- new net N$78: IC5C.O, IC8A.ENC
- new net N$79: IC7B.I
- net CHANGE_CLOCK_SELECT: now also IC5C.I0, IC7D.I; no longer IC1D.I1, IC4A.D, IC8A.ENC
- net GND: now also C24.2, S14.P, S14.P1; no longer IC10A.I0, IC10A.I1, IC5B.I, IC5C.I, IC5D.I, IC5E.I, S1.P, S1.P1
- net N$1: now also IC5B.I0; no longer IC1B.I0
- net N$10: now also IC4A.D, IC5D.I1, IC7D.O, IC7F.I; no longer IC4B.D, IC5F.O
- net N$2: now also IC7B.O; no longer IC1A.I1, IC1C.O
- net N$4: now also IC4B.D, IC5D.O; no longer IC1D.O, IC5F.I
- net N$5: now also IC2A.W, IC4A.CLK, IC4B.CLK; no longer IC1A.I0, IC1C.I1, R27.1, S1.S, S1.S1
- net N$8: now also IC5D.I0; no longer IC1D.I0
- net N$9: now also IC7A.I, IC7F.O; no longer IC4A.CLK, IC4B.CLK, IC5A.O
- net RING_CNTR_CLOCK: now also IC5B.O; no longer IC1B.O
- net SELECTED_CLOCK: now also IC5B.I1; no longer IC1B.I1, IC5A.I
- net SINGLE_STEP_CLOCK: now also IC7C.O; no longer IC1A.O, IC1C.I0
- net VCC: now also R2.2; no longer R27.2
Other:
- note added: "373 needs to be edge triggered"
- note added: "Achtung, SchmittTigger noch nicht verbaut. Noch ist da ein normaler Inverter. Muss noch bestellt werden"
- note removed: "maybe need some time delay here"
- moved on the sheet: C2, C3, C4, C5, C6, C7, C8, C9, IC10B, IC10C, IC10D, IC11A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

Commit message: finished and tested ui-board.
I Didnt check all clocks. 16Mhz, 4Mhz and the single_clock work
Connections:
- net 31.25KHZ renamed 250KHZ
- removed net 500KHZ: IC13A.QD, IC13B.A, IC2A.D2, JP4.7
- removed net N$2: IC7B.O
- removed net N$67: IC7E.O
- removed net N$77: IC7E.I
- removed net N$79: IC7B.I
- new net 16MHZ: IC13A.A, IC2A.D6, QG2.OUT
- net 1MHZ: now also IC13A.QD, IC13B.A, IC2A.D2, JP4.7; no longer IC13A.QC, IC2A.D3, JP4.5
- net 2MHZ: now also IC13A.QC, IC2A.D3, JP4.5; no longer IC13A.QB, IC2A.D4, JP4.3
- net 4MHZ: now also IC13A.QB, IC2A.D4, JP4.3; no longer IC13A.QA, IC2A.D5, JP4.1
- net 8MHZ: now also IC13A.QA, IC2A.D5, JP4.1; no longer IC13A.A, IC2A.D6, QG2.OUT
Other:
- note removed: "Achtung, SchmittTigger noch nicht verbaut. Noch ist da ein normaler Inverter. Muss noch bestellt werden"
- moved on the sheet: C13, C14, C15, C16, C17, C18, C19, C20, C21, C22, C23, C24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
